File: solar-glow-drh-v1.kicad_pcb (KiCad board)
At the start: 2 copper layers, 50.8 x 88.9 mm, 0 parts

Commit message: Add files via upload
Parts:
- added MH1: , MountingHole_M2_2.2mm, F.Cu at (3.50, 85.9)
- added MH2: , MountingHole_M2_2.2mm, F.Cu at (47.3, 85.9)
- added MH3: , MountingHole_M2_2.2mm, F.Cu at (3.50, 29.9)
- added MH4: , MountingHole_M2_2.2mm, F.Cu at (47.3, 29.9)

Commit message: Add files via upload
Parts:
- added C1: 100nF, 100nF, B.Cu at (14.3, 38.3)
- added C2: cap, cap, B.Cu at (8.00, 85.3)
- added C3: cap, cap, B.Cu at (41.0, 85.3)
- added C4: cap, cap, B.Cu at (38.5, 38.3)
- added D1: SOD-123, SOD-123, B.Cu at (18.0, 85.3)
- added D2: LA P47F, LA_P47F, B.Cu at (16.1, 43.9)
- added D3: LA P47F, LA_P47F, B.Cu at (22.4, 43.9)
- added D4: LA P47F, LA_P47F, B.Cu at (28.7, 43.9)
- added D5: LA P47F, LA_P47F, B.Cu at (34.7, 43.9)
- added D6: SOD-523, SOD-523, B.Cu at (25.4, 26.9)
- added D7: SOD-523, SOD-523, B.Cu at (25.4, 14.9)
- added J1: UPDI, UPDI, B.Cu at (5.60, 38.3)
- added JP1: I2C, I2C, B.Cu at (18.2, 38.3)
- added R1: 1k, 1k, B.Cu at (16.1, 49.6)
- added R2: 1k, 1k, B.Cu at (22.4, 49.6)
- added R3: 1k, 1k, B.Cu at (28.7, 49.6)
- added R4: 1k, 1k, B.Cu at (34.7, 49.6)
- added SC1: WS17 1F, WS17_1F, B.Cu at (15.5, 21.4)
- added SC2: WS17 1F, WS17_1F, B.Cu at (35.3, 21.4)
- added SC3: WS17 1F, WS17_1F, B.Cu at (15.5, 67.5)
- added SC4: WS17 1F, WS17_1F, B.Cu at (35.3, 67.5)
- added SW2: slide OFF/ON/TINY, slide_OFF/ON/TINY, B.Cu at (28.5, 85.3)
- added TC1: Tag-Connect, TC2030-IDC-NL, B.Cu at (15.5, 21.4)
- added U1: AVR64DD28, AVR64DD28, B.Cu at (10.6, 38.3)
- added U2: ALD910025, ALD910025, B.Cu at (31.0, 38.3)
Other:
- rule pad_to_mask_clearance: 0.0 -> 0

Commit message: Add files via upload
Parts:
- moved TC1 4.00 mm to (11.5, 21.4)
Changed lines of the file:
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@@
   )
   (footprint "TC2030-IDC-NL" (layer "B.Cu")
-    (at 15.5 21.4)
+    (at 11.5 21.4)
     (attr smd exclude_from_bom)
-    (fp_rect (start -3.0 -4.95) (end 3.0 4.95) (layer "B.CrtYd") (width 0.05) (fill none))
+    (fp_rect (start -3 -4.95) (end 3 4.95) (layer "B.CrtYd") (width 0.05) (fill none))
     (fp_text reference "TC1" (at 0 0 0) (layer "B.SilkS")
       (effects (font (size 0.7 0.7) (thickness 0.12)))

Commit message: Add files via upload
Other:
- copper layers 2 -> 4
Changed lines of the file:
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@@
 (kicad_pcb (version 20211014) (generator kiutils)
   (general
-    (thickness 1.6)
+    (thickness 0.4)
   )
   (paper "A4")
   (layers
     (0 "F.Cu" signal)
+    (1 "In1.Cu" signal "GND.plane")
+    (2 "In2.Cu" signal "VS.plane")
     (31 "B.Cu" signal)
     (32 "B.Adhes" user "B.Adhesive")

Commit message: Add files via upload
Parts:
- C1: value 100nF -> (none); footprint 100nF -> C1:0805
- C2: value cap -> (none); footprint cap -> C2:0805
- C3: value cap -> (none); footprint cap -> C3:0805
- C4: value cap -> (none); footprint cap -> C4:0402
- D1: value SOD-123 -> (none); footprint SOD-123 -> D1:SOD
- D2: value LA P47F -> (none); footprint LA_P47F -> D2:LED
- D3: value LA P47F -> (none); footprint LA_P47F -> D3:LED
- D4: value LA P47F -> (none); footprint LA_P47F -> D4:LED
- D5: value LA P47F -> (none); footprint LA_P47F -> D5:LED
- D6: value SOD-523 -> (none); footprint SOD-523 -> D6:SOD
- D7: value SOD-523 -> (none); footprint SOD-523 -> D7:SOD
- J1: value UPDI -> (none); footprint UPDI -> J1:PROG
- JP1: value I2C -> (none); footprint I2C -> JP1:PROG
- R1: value 1k -> (none); footprint 1k -> R1:0402
- R2: value 1k -> (none); footprint 1k -> R2:0402
- R3: value 1k -> (none); footprint 1k -> R3:0402
- R4: value 1k -> (none); footprint 1k -> R4:0402
- SC1: value WS17 1F -> (none); footprint WS17_1F -> SC1:SCPC
- SC2: value WS17 1F -> (none); footprint WS17_1F -> SC2:SCPC
- SC3: value WS17 1F -> (none); footprint WS17_1F -> SC3:SCPC
- SC4: value WS17 1F -> (none); footprint WS17_1F -> SC4:SCPC
- U1: value AVR64DD28 -> (none); footprint AVR64DD28 -> U1:QFN28
- U2: value ALD910025 -> (none); footprint ALD910025 -> U2:SOIC8
- turned D6 to 90 degrees
- turned D7 to 90 degrees
- turned SC1 to 270 degrees
- turned SC2 to 90 degrees
- turned SC3 to 270 degrees
- turned SC4 to 90 degrees
Connections:
- C1 pad 1: (no net) -> VS
- C1 pad 2: (no net) -> GND
- C2 pad 1: (no net) -> VS
- C2 pad 2: (no net) -> GND
- C3 pad 1: (no net) -> VDDIO2
- C3 pad 2: (no net) -> GND
- C4 pad 1: (no net) -> VS
- C4 pad 2: (no net) -> GND
- R1 pad 1: (no net) -> K2
- R1 pad 2: (no net) -> LDRV1
- R2 pad 1: (no net) -> K3
- R2 pad 2: (no net) -> LDRV2
- R3 pad 1: (no net) -> K4
- R3 pad 2: (no net) -> LDRV3
- R4 pad 1: (no net) -> K5
- R4 pad 2: (no net) -> LDRV4
- TC1 pad 1: (no net) -> UPDI
- TC1 pad 2: (no net) -> VS
- TC1 pad 3: (no net) -> GND

Commit message: Add files via upload
Parts:
- turned SC1 to 90 degrees
- turned SC2 to 270 degrees
Changed lines of the file:
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@@
   )
   (footprint "SC1:SCPC" (layer "B.Cu")
-    (at 15.5 21.4 270)
+    (at 15.5 21.4 90)
     (attr smd)
     (fp_rect (start -14.25 -8.5) (end 14.25 8.5) (layer "B.CrtYd") (width 0.05) (fill none))
@@
       (effects (font (size 0.6 0.6) (thickness 0.1)))
     )
-    (pad "P" smd roundrect (at 16.5 -6.25) (size 3.5 3.5) (layers "B.Cu" "B.Mask" "B.Paste") (roundrect_rratio 0.2)
+    (pad "P" smd roundrect (at -11 0) (size 3.5 7.75) (layers "B.Cu" "B.Mask" "B.Paste") (roundrect_rratio 0.2)
       (net 22 "VS"))
-    (pad "N" smd roundrect (at -16.5 6.25) (size 3.5 3.5) (layers "B.Cu" "B.Mask" "B.Paste") (roundrect_rratio 0.2)
+    (pad "N" smd roundrect (at 11 0) (size 3.5 12.25) (layers "B.Cu" "B.Mask" "B.Paste") (roundrect_rratio 0.2)
       (net 12 "MID"))
   )
   (footprint "SC2:SCPC" (layer "B.Cu")
-    (at 35.3 21.4 90)
+    (at 35.3 21.4 270)
     (attr smd)
     (fp_rect (start -14.25 -8.5) (end 14.25 8.5) (layer "B.CrtYd") (width 0.05) (fill none))
@@
       (effects (font (size 0.6 0.6) (thickness 0.1)))
     )
-    (pad "P" smd roundrect (at 16.5 -6.25) (size 3.5 3.5) (layers "B.Cu" "B.Mask" "B.Paste") (roundrect_rratio 0.2)
+    (pad "P" smd roundrect (at -11 0) (size 3.5 7.75) (layers "B.Cu" "B.Mask" "B.Paste") (roundrect_rratio 0.2)
       (net 12 "MID"))
-    (pad "N" smd roundrect (at -16.5 6.25) (size 3.5 3.5) (layers "B.Cu" "B.Mask" "B.Paste") (roundrect_rratio 0.2)
+    (pad "N" smd roundrect (at 11 0) (size 3.5 12.25) (layers "B.Cu" "B.Mask" "B.Paste") (roundrect_rratio 0.2)
       (net 1 "GND"))
   )
@@
       (effects (font (size 0.6 0.6) (thickness 0.1)))
     )
-    (pad "P" smd roundrect (at 16.5 -6.25) (size 3.5 3.5) (layers "B.Cu" "B.Mask" "B.Paste") (roundrect_rratio 0.2)
+    (pad "P" smd roundrect (at -11 0) (size 3.5 7.75) (layers "B.Cu" "B.Mask" "B.Paste") (roundrect_rratio 0.2)
       (net 22 "VS"))
-    (pad "N" smd roundrect (at -16.5 6.25) (size 3.5 3.5) (layers "B.Cu" "B.Mask" "B.Paste") (roundrect_rratio 0.2)
+    (pad "N" smd roundrect (at 11 0) (size 3.5 12.25) (layers "B.Cu" "B.Mask" "B.Paste") (roundrect_rratio 0.2)
       (net 12 "MID"))
   )
@@
       (effects (font (size 0.6 0.6) (thickness 0.1)))
     )
-    (pad "P" smd roundrect (at 16.5 -6.25) (size 3.5 3.5) (layers "B.Cu" "B.Mask" "B.Paste") (roundrect_rratio 0.2)
+    (pad "P" smd roundrect (at -11 0) (size 3.5 7.75) (layers "B.Cu" "B.Mask" "B.Paste") (roundrect_rratio 0.2)
       (net 12 "MID"))
-    (pad "N" smd roundrect (at -16.5 6.25) (size 3.5 3.5) (layers "B.Cu" "B.Mask" "B.Paste") (roundrect_rratio 0.2)
+    (pad "N" smd roundrect (at 11 0) (size 3.5 12.25) (layers "B.Cu" "B.Mask" "B.Paste") (roundrect_rratio 0.2)
       (net 1 "GND"))
   )

Commit message: Add files via upload
Parts:
- added BT1: , BT1:RTNR, F.Cu at (17.4, 15.9)
- added BT2: , BT2:RTNR, F.Cu at (33.4, 15.9)
- added C5: , C5:0402, B.Cu at (13.5, 41.4)
- added PV1: , PV1:SOLAR, F.Cu at (25.4, 15.9)
- added R5: , R5:0402, B.Cu at (9.50, 41.4)
- added R6: , R6:0402, B.Cu at (11.5, 41.4)
- added SJ1: , SJ1:0402, B.Cu at (7.00, 41.4)
- added SW1: SW_F12340, SW1:SW_F12340, F.Cu at (40.4, 77.9)

Commit message: Add files via upload
Parts:
- moved C3 50.5 mm to (12.0, 43.9)
- moved D1 48.9 mm to (44.0, 43.9)
- moved C2 47.4 mm to (8.00, 37.9)
- moved U2 12.1 mm to (43.0, 39.9)
- moved C1 10.9 mm to (5.00, 43.9)
- moved C4 9.14 mm to (47.5, 39.9)
- moved C5 7.91 mm to (7.00, 45.9)
- moved R5 7.91 mm to (3.00, 45.9)
- moved R6 7.91 mm to (5.00, 45.9)
- moved SJ1 6.02 mm to (13.0, 41.9)
- moved JP1 4.72 mm to (13.5, 37.9), turned to 90 degrees
- moved SW2 3.52 mm to (25.0, 84.9)
- moved U1 2.82 mm to (9.50, 40.9)
- moved J1 2.63 mm to (3.00, 37.9), turned to 90 degrees
Changed lines of the file:
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@@
   )
   (footprint "slide_OFF/ON/TINY" (layer "B.Cu")
-    (at 28.5 85.3)
+    (at 25.0 84.9 0)
     (attr smd)
     (fp_rect (start -3.3 -1.5) (end 3.3 1.5) (layer "B.CrtYd") (width 0.05) (fill none))
@@
   )
   (footprint "U1:QFN28" (layer "B.Cu")
-    (at 10.6 38.3 0)
+    (at 9.5 40.9 0)
     (attr smd)
     (fp_rect (start -2 -2) (end 2 2) (layer "B.CrtYd") (width 0.05) (fill none))
@@
   )
   (footprint "U2:SOIC8" (layer "B.Cu")
-    (at 31 38.3 0)
+    (at 43.0 39.9 0)
     (attr smd)
     (fp_rect (start -2.45 -1.95) (end 2.45 1.95) (layer "B.CrtYd") (width 0.05) (fill none))
@@
   )
   (footprint "D1:SOD" (layer "B.Cu")
-    (at 18 85.3 0)
+    (at 44.0 43.9 0)
     (attr smd)
     (fp_rect (start -1.85 -0.8) (end 1.85 0.8) (layer "B.CrtYd") (width 0.05) (fill none))
@@
   )
   (footprint "C1:0805" (layer "B.Cu")
-    (at 14.3 38.3 0)
+    (at 5.0 43.9 0)
     (attr smd)
     (fp_rect (start -1 -0.625) (end 1 0.625) (layer "B.CrtYd") (width 0.05) (fill none))
@@
   )
   (footprint "C2:0805" (layer "B.Cu")
-    (at 8 85.3 0)
+    (at 8.0 37.9 0)
     (attr smd)
     (fp_rect (start -1 -0.625) (end 1 0.625) (layer "B.CrtYd") (width 0.05) (fill none))
@@
   )
   (footprint "C3:0805" (layer "B.Cu")
-    (at 41 85.3 0)
+    (at 12.0 43.9 0)
     (attr smd)
     (fp_rect (start -1 -0.625) (end 1 0.625) (layer "B.CrtYd") (width 0.05) (fill none))
@@
   )
   (footprint "C4:0402" (layer "B.Cu")
-    (at 38.5 38.3 0)
+    (at 47.5 39.9 0)
     (attr smd)
     (fp_rect (start -0.5 -0.25) (end 0.5 0.25) (layer "B.CrtYd") (width 0.05) (fill none))
@@
   )
   (footprint "J1:PROG" (layer "B.Cu")
-    (at 5.6 38.3 0)
+    (at 3.0 37.9 90)
     (attr smd)
     (fp_text reference "J1" (at 0 0 0) (layer "B.SilkS")
@@
   )
   (footprint "JP1:PROG" (layer "B.Cu")
-    (at 18.2 38.3 0)
+    (at 13.5 37.9 90)
     (attr smd)
     (fp_text reference "JP1" (at 0 0 0) (layer "B.SilkS")
@@
   )
   (footprint "SJ1:0402" (layer "B.Cu")
-    (at 7.0 41.4 0)
+    (at 13.0 41.9 0)
     (attr smd)
     (fp_rect (start -0.5 -0.25) (end 0.5 0.25) (layer "B.CrtYd") (width 0.05) (fill none))
@@
   )
   (footprint "R5:0402" (layer "B.Cu")
-    (at 9.5 41.4 0)
+    (at 3.0 45.9 0)
     (attr smd)
     (fp_rect (start -0.5 -0.25) (end 0.5 0.25) (layer "B.CrtYd") (width 0.05) (fill none))
@@
   )
   (footprint "R6:0402" (layer "B.Cu")
-    (at 11.5 41.4 0)
+    (at 5.0 45.9 0)
     (attr smd)
     (fp_rect (start -0.5 -0.25) (end 0.5 0.25) (layer "B.CrtYd") (width 0.05) (fill none))
@@
   )
   (footprint "C5:0402" (layer "B.Cu")
-    (at 13.5 41.4 0)
-    (attr smd)
-    (fp_rect (start -0.5 -0.25) (end 0.5 0.25) (layer "B.CrtYd") (width 0.05) (fill none))
+    (at 7.0 45.9 0)
+    (attr smd)
+    (fp_rect (start -0.5 -0.25) (end 0.5 0.25) (layer "B.CrtYd") (width 0.05) (fill none))
