File: solar-glow-drh-v2_1.kicad_pcb (KiCad board)
At the start: 6 copper layers, 50.8 x 88.9 mm, 51 parts

Commit message: Add files via upload
Connections:
- U1 pad 12: (no net) -> VSENSE
- U1 pad 5: VSENSE -> (no net)
Routing:
- net SDA: track 27.8 -> 32.0 mm
- net VSENSE: track 14.2 -> 15.6 mm
- net VDDIO2: track 13.7 -> 14.4 mm

Commit message: Add files via upload
Parts:
- C1, C2, C3, C4, C6, C7: value (none) -> 100nF
- C5: value (none) -> VSENSE filt
- D1, D9: value (none) -> MMSD301T1G
- D2, D3, D4, D5: value (none) -> LA P47F
- J1: value (none) -> UPDI hdr
- JP1: value (none) -> I2C brk
- JP2: value (none) -> GPIO brk
- MH1, MH2, MH3, MH4: value (none) -> M2
- PV1, PV2: value (none) -> SM141K06L
- Q1: value (none) -> BCP5316MTWG
- R1, R2, R3, R4: value (none) -> LED ballast
- R10, R11: value (none) -> 4.7k
- R12: value (none) -> TINY ballast
- R5, R6: value (none) -> VSENSE div
- R7: value (none) -> 1.8M
- R8: value (none) -> 1M
- R9: value (none) -> 1k
- SB1: value (none) -> LED1 jmp
- SB2: value (none) -> LED2 jmp
- SB3: value (none) -> LED3 jmp
- SB4: value (none) -> LED4 jmp
- SC1, SC2, SC3, SC4: value (none) -> WS17 1F 2.75V
- SJ1: value (none) -> VDDIO2 jmp
- SW2: value (none) -> LED master
- TC1: value (none) -> Tag-Connect
- U1: value (none) -> AVR64DD28 (VQFN28)
- U2: value (none) -> ALD910025SAL
- U3: value (none) -> LIS2DH12
- U4: value (none) -> TLV431BCDBZR
Connections:
- TC1 pad 4: (no net) -> unconnected-(TC1-Pad4)
- TC1 pad 5: (no net) -> unconnected-(TC1-Pad5)
- TC1 pad 6: (no net) -> unconnected-(TC1-Pad6)
- U1 pad 11: (no net) -> unconnected-(U1-PD1-Pad11)
- U1 pad 13: (no net) -> unconnected-(U1-PD3-Pad13)
- U1 pad 14: (no net) -> unconnected-(U1-PD4-Pad14)
- U1 pad 15: (no net) -> unconnected-(U1-PD5-Pad15)
- U1 pad 16: (no net) -> unconnected-(U1-PD6-Pad16)
- U1 pad 17: (no net) -> unconnected-(U1-PD7-Pad17)
- U1 pad 22: (no net) -> unconnected-(U1-PF6/RST-Pad22)
- U1 pad 4: (no net) -> unconnected-(U1-PA6-Pad4)
- U1 pad 5: (no net) -> unconnected-(U1-PA7-Pad5)
Other:
- board text added: "GND"
- board text added: "OFF"
- board text added: "ON"
- board text added: "PA4"
- board text added: "PC0"
- board text added: "PC1"
- board text added: "SCL"
- board text added: "SDA"
- board text added: "TINY"
- board text added: "UPDI"
- board text added: "VS"
