File: solar-glow-drh-v2_1.kicad_pcb (KiCad board)
At the start: 6 copper layers, 50.8 x 88.9 mm, 51 parts, among them J1 UPDI hdr, Q1 BCP5316MTWG, SW2 LED master, U1 AVR64DD28 (VQFN28), U2 ALD910025SAL, U3 LIS2DH12, U4 TLV431BCDBZR

Commit message: Add files via upload
Parts:
- moved U2 14.8 mm to (28.5, 37.0)
Routing:
- net MID: track 105.2 -> 126.1 mm
Changed lines of the file:
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@@
 		(at 13.3 46)
 		(property "Reference" "SJ1"
-			(at -0.4373 -2.2402 0.0)
+			(at -0.89 -2.64 0.0)
 			(layer "B.SilkS")
 			(effects
@@
 	(footprint "solarglow:U2"
 		(layer "B.Cu")
-		(at 43 39.9)
+		(at 28.5 37)
 		(property "Reference" "U2"
 			(at -4.475 0.0 0.0)
@@
 	)
 	(via
-		(at 45.6 41.805)
+		(at 31.1 38.9)
 		(size 0.6)
 		(drill 0.3)
@@
 	)
 	(via
-		(at 40.4 37.995)
+		(at 25.9 35.09)
 		(size 0.6)
 		(drill 0.3)
@@
 	)
 	(via
-		(at 40.4 41.8)
+		(at 25.9 38.9)
 		(size 0.4)
 		(drill 0.2)
@@
 	)
 	(via
-		(at 45.6 40.5)
+		(at 31.1 37.63)
 		(size 0.4)
 		(drill 0.2)
@@
 	)
 	(segment
-		(start 45.6 40.535)
-		(end 45.6 39.265)
-		(width 0.22)
-		(layer "B.Cu")
-		(net "MID")
-	)
-	(segment
 		(start 40.4 45)
 		(end 47 45)
@@
 	)
 	(segment
-		(start 47 40.5)
-		(end 45.6 40.535)
-		(width 0.22)
-		(layer "In2.Cu")
-		(net "MID")
-	)
-	(segment
 		(start 38.5 41.8)
 		(end 40.4 41.805)
@@
 	(segment
 		(start 47 45)
-		(end 47 40.5)
-		(width 0.22)
-		(layer "In2.Cu")
-		(net "MID")
-	)
-	(segment
-		(start 47 45)
 		(end 47 61)
 		(width 0.22)
@@
 	)
 	(via
-		(at 40.4 39.265)
+		(at 25.9 36.37)
 		(size 0.6)
 		(drill 0.3)
@@
 	)
 	(via
-		(at 40.4 40.535)
+		(at 25.9 37.63)
 		(size 0.6)
 		(drill 0.3)
@@
 	)
 	(via
-		(at 45.6 37.995)
+		(at 31.1 35.09)
 		(size 0.6)
 		(drill 0.3)
@@
 		(layer "B.Mask")
 	)
+	(segment
+		(start 25.9 38.9)
+		(end 25.0 38.9)
+		(width 0.22)
+		(layer "In2.Cu")
+		(net "MID")
+	)
+	(segment
+		(start 25.0 38.9)
+		(end 25.0 26.0)
+		(width 0.22)
+		(layer "In2.Cu")
+		(net "MID")
+	)
+	(segment
+		(start 31.1 37.63)
+		(end 32.5 37.63)
+		(width 0.22)
+		(layer "In2.Cu")
+		(net "MID")
+	)
+	(segment
+		(start 32.5 37.63)
+		(end 32.5 26.0)
+		(width 0.22)
+		(layer "In2.Cu")
+		(net "MID")
+	)
+	(segment
+		(start 31.1 37.63)
+		(end 31.1 36.37)
+		(width 0.22)
+		(layer "B.Cu")
+		(net "MID")
+	)
+	(gr_poly (pts
+				(xy 46.2500 40.5000)
+				(xy 46.2337 40.6446)
+				(xy 46.1856 40.7820)
+				(xy 46.1082 40.9053)
+				(xy 46.0053 41.0082)
+				(xy 45.8820 41.0856)
+				(xy 45.7446 41.1337)
+				(xy 45.6000 41.1500)
+				(xy 45.4554 41.1337)
+				(xy 45.3180 41.0856)
+				(xy 45.1947 41.0082)
+				(xy 45.0918 40.9053)
+				(xy 45.0144 40.7820)
+				(xy 44.9663 40.6446)
+				(xy 44.9500 40.5000)
+				(xy 44.9663 40.3554)
+				(xy 45.0144 40.2180)
+				(xy 45.0918 40.0947)
+				(xy 45.1947 39.9918)
+				(xy 45.3180 39.9144)
+				(xy 45.4554 39.8663)
+				(xy 45.6000 39.8500)
+				(xy 45.7446 39.8663)
+				(xy 45.8820 39.9144)
+				(xy 46.0053 39.9918)
+				(xy 46.1082 40.0947)
+				(xy 46.1856 40.2180)
+				(xy 46.2337 40.3554)
+			) (stroke (width 0) (type solid)) (fill solid) (layer "F.Cu"))
+	(gr_poly (pts
+				(xy 41.0500 40.5300)
+				(xy 41.0337 40.6746)
+				(xy 40.9856 40.8120)
+				(xy 40.9082 40.9353)
+				(xy 40.8053 41.0382)
+				(xy 40.6820 41.1156)
+				(xy 40.5446 41.1637)
+				(xy 40.4000 41.1800)
+				(xy 40.2554 41.1637)
+				(xy 40.1180 41.1156)
+				(xy 39.9947 41.0382)
+				(xy 39.8918 40.9353)
+				(xy 39.8144 40.8120)
+				(xy 39.7663 40.6746)
+				(xy 39.7500 40.5300)
+				(xy 39.7663 40.3854)
+				(xy 39.8144 40.2480)
+				(xy 39.8918 40.1247)
+				(xy 39.9947 40.0218)
+				(xy 40.1180 39.9444)
+				(xy 40.2554 39.8963)
+				(xy 40.4000 39.8800)
+				(xy 40.5446 39.8963)
+				(xy 40.6820 39.9444)
+				(xy 40.8053 40.0218)
+				(xy 40.9082 40.1247)
+				(xy 40.9856 40.2480)
+				(xy 41.0337 40.3854)
+			) (stroke (width 0) (type solid)) (fill solid) (layer "F.Cu"))
+	(gr_poly (pts
+				(xy 41.0500 41.8000)
+				(xy 41.0337 41.9446)
+				(xy 40.9856 42.0820)
+				(xy 40.9082 42.2053)
+				(xy 40.8053 42.3082)
+				(xy 40.6820 42.3856)
+				(xy 40.5446 42.4337)
+				(xy 40.4000 42.4500)
+				(xy 40.2554 42.4337)
+				(xy 40.1180 42.3856)
+				(xy 39.9947 42.3082)
+				(xy 39.8918 42.2053)
+				(xy 39.8144 42.0820)
+				(xy 39.7663 41.9446)
+				(xy 39.7500 41.8000)
+				(xy 39.7663 41.6554)
+				(xy 39.8144 41.5180)
+				(xy 39.8918 41.3947)
+				(xy 39.9947 41.2918)
+				(xy 40.1180 41.2144)
+				(xy 40.2554 41.1663)
+				(xy 40.4000 41.1500)
+				(xy 40.5446 41.1663)
+				(xy 40.6820 41.2144)
+				(xy 40.8053 41.2918)
+				(xy 40.9082 41.3947)
+				(xy 40.9856 41.5180)
+				(xy 41.0337 41.6554)
+			) (stroke (width 0) (type solid)) (fill solid) (layer "F.Cu"))
+	(gr_poly (pts
+				(xy 46.2500 41.8000)
+				(xy 46.2337 41.9446)
+				(xy 46.1856 42.0820)
+				(xy 46.1082 42.2053)
+				(xy 46.0053 42.3082)
+				(xy 45.8820 42.3856)
+				(xy 45.7446 42.4337)
+				(xy 45.6000 42.4500)
+				(xy 45.4554 42.4337)
+				(xy 45.3180 42.3856)
+				(xy 45.1947 42.3082)
+				(xy 45.0918 42.2053)
+				(xy 45.0144 42.0820)
+				(xy 44.9663 41.9446)
+				(xy 44.9500 41.8000)
+				(xy 44.9663 41.6554)
+				(xy 45.0144 41.5180)
+				(xy 45.0918 41.3947)
+				(xy 45.1947 41.2918)
+				(xy 45.3180 41.2144)
+				(xy 45.4554 41.1663)
+				(xy 45.6000 41.1500)
+				(xy 45.7446 41.1663)
+				(xy 45.8820 41.2144)
+				(xy 46.0053 41.2918)
+				(xy 46.1082 41.3947)
+				(xy 46.1856 41.5180)
+				(xy 46.2337 41.6554)
+			) (stroke (width 0) (type solid)) (fill solid) (layer "F.Cu"))
 )

Commit message: Add files via upload
Routing:
- net VS: track 19.9 -> 26.8 mm
- net VIN: track 90.2 -> 94.1 mm
Changed lines of the file:
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@@
 	)
 	(via
-		(at 44.8 43.5)
-		(size 0.6)
-		(drill 0.3)
-		(layers "F.Cu" "B.Cu")
-		(capping no)
-		(covering
-			(front yes)
-			(back no)
-		)
-		(plugging
-			(front no)
-			(back no)
-		)
-		(filling no)
-		(net "VIN")
-	)
-	(via
 		(at 3.69 50.4)
 		(size 0.6)
@@
 	)
 	(segment
-		(start 44.8 43.5)
-		(end 45.85 43.9)
-		(width 0.22)
-		(layer "B.Cu")
-		(net "VIN")
-	)
-	(segment
 		(start 44.8 28)
 		(end 44.8 43.5)
@@
 	)
 	(via
-		(at 45.5 46.13)
-		(size 0.6)
-		(drill 0.3)
-		(layers "F.Cu" "B.Cu")
-		(capping no)
-		(covering
-			(front no)
-			(back no)
-		)
-		(plugging
-			(front no)
-			(back no)
-		)
-		(filling no)
-		(net "VS")
-	)
-	(via
 		(at 33.52 48.6)
 		(size 0.6)
@@
 	)
 	(via
-		(at 42.15 42.88)
-		(size 0.6)
-		(drill 0.3)
-		(layers "F.Cu" "B.Cu")
-		(capping no)
-		(covering
-			(front yes)
-			(back no)
-		)
-		(plugging
-			(front no)
-			(back no)
-		)
-		(filling no)
-		(net "VS")
-	)
-	(via
 		(at 15.5 83)
 		(size 0.6)
@@
 	)
 	(segment
-		(start 45.5 47.05)
-		(end 45.5 46.13)
-		(width 0.22)
-		(layer "B.Cu")
-		(net "VS")
-	)
-	(segment
 		(start 32.5 48.6)
 		(end 33.52 48.6)
@@
 	)
 	(segment
-		(start 42.15 43.9)
-		(end 42.15 42.88)
-		(width 0.22)
-		(layer "B.Cu")
-		(net "VS")
-	)
-	(segment
 		(start 41.5 49.5)
 		(end 41.5 51)
@@
 				(xy 46.2337 41.6554)
 			) (stroke (width 0) (type solid)) (fill solid) (layer "F.Cu"))
+	(via
+		(at 44.8 39.0)
+		(size 0.6)
+		(drill 0.3)
+		(layers "F.Cu" "B.Cu")
+		(capping no)
+		(covering
+			(front yes)
+			(back no)
+		)
+		(plugging
+			(front no)
+			(back no)
+		)
+		(filling no)
+		(net "VIN")
+	)
+	(via
+		(at 42.15 39.0)
+		(size 0.6)
+		(drill 0.3)
+		(layers "F.Cu" "B.Cu")
+		(capping no)
+		(covering
+			(front yes)
+			(back no)
+		)
+		(plugging
+			(front no)
+			(back no)
+		)
+		(filling no)
+		(net "VS")
+	)
+	(via
+		(at 49.4 47.05)
+		(size 0.6)
+		(drill 0.3)
+		(layers "F.Cu" "B.Cu")
+		(capping no)
+		(covering
+			(front yes)
+			(back no)
+		)
+		(plugging
+			(front no)
+			(back no)
+		)
+		(filling no)
+		(net "VS")
+	)
+	(segment
+		(start 45.85 43.9)
+		(end 44.8 39.0)
+		(width 0.22)
+		(layer "B.Cu")
+		(net "VIN")
+	)
+	(segment
+		(start 42.15 43.9)
+		(end 42.15 39.0)
+		(width 0.22)
+		(layer "B.Cu")
+		(net "VS")
+	)
+	(segment
+		(start 45.5 47.05)
+		(end 49.4 47.05)
+		(width 0.22)
+		(layer "B.Cu")
+		(net "VS")
+	)
+	(gr_poly (pts
+				(xy 45.4500 43.5000)
+				(xy 45.4337 43.6446)
+				(xy 45.3856 43.7820)
+				(xy 45.3082 43.9053)
+				(xy 45.2053 44.0082)
+				(xy 45.0820 44.0856)
+				(xy 44.9446 44.1337)
+				(xy 44.8000 44.1500)
+				(xy 44.6554 44.1337)
+				(xy 44.5180 44.0856)
+				(xy 44.3947 44.0082)
+				(xy 44.2918 43.9053)
+				(xy 44.2144 43.7820)
+				(xy 44.1663 43.6446)
+				(xy 44.1500 43.5000)
+				(xy 44.1663 43.3554)
+				(xy 44.2144 43.2180)
+				(xy 44.2918 43.0947)
+				(xy 44.3947 42.9918)
+				(xy 44.5180 42.9144)
+				(xy 44.6554 42.8663)
+				(xy 44.8000 42.8500)
+				(xy 44.9446 42.8663)
+				(xy 45.0820 42.9144)
+				(xy 45.2053 42.9918)
+				(xy 45.3082 43.0947)
+				(xy 45.3856 43.2180)
+				(xy 45.4337 43.3554)
+			) (stroke (width 0) (type solid)) (fill solid) (layer "F.Cu"))
+	(gr_poly (pts
+				(xy 42.8000 42.8800)
+				(xy 42.7837 43.0246)
+				(xy 42.7356 43.1620)
+				(xy 42.6582 43.2853)
+				(xy 42.5553 43.3882)
+				(xy 42.4320 43.4656)
+				(xy 42.2946 43.5137)
+				(xy 42.1500 43.5300)
+				(xy 42.0054 43.5137)
+				(xy 41.8680 43.4656)
+				(xy 41.7447 43.3882)
+				(xy 41.6418 43.2853)
+				(xy 41.5644 43.1620)
+				(xy 41.5163 43.0246)
+				(xy 41.5000 42.8800)
+				(xy 41.5163 42.7354)
+				(xy 41.5644 42.5980)
+				(xy 41.6418 42.4747)
+				(xy 41.7447 42.3718)
+				(xy 41.8680 42.2944)
+				(xy 42.0054 42.2463)
+				(xy 42.1500 42.2300)
+				(xy 42.2946 42.2463)
+				(xy 42.4320 42.2944)
+				(xy 42.5553 42.3718)
+				(xy 42.6582 42.4747)
+				(xy 42.7356 42.5980)
+				(xy 42.7837 42.7354)
+			) (stroke (width 0) (type solid)) (fill solid) (layer "F.Cu"))
+	(gr_poly (pts
+				(xy 46.1500 46.1300)
+				(xy 46.1337 46.2746)
+				(xy 46.0856 46.4120)
+				(xy 46.0082 46.5353)
+				(xy 45.9053 46.6382)
+				(xy 45.7820 46.7156)
+				(xy 45.6446 46.7637)
+				(xy 45.5000 46.7800)
+				(xy 45.3554 46.7637)
+				(xy 45.2180 46.7156)
+				(xy 45.0947 46.6382)
+				(xy 44.9918 46.5353)
+				(xy 44.9144 46.4120)
+				(xy 44.8663 46.2746)
+				(xy 44.8500 46.1300)
+				(xy 44.8663 45.9854)
+				(xy 44.9144 45.8480)
+				(xy 44.9918 45.7247)
+				(xy 45.0947 45.6218)
+				(xy 45.2180 45.5444)
+				(xy 45.3554 45.4963)
+				(xy 45.5000 45.4800)
+				(xy 45.6446 45.4963)
+				(xy 45.7820 45.5444)
+				(xy 45.9053 45.6218)
+				(xy 46.0082 45.7247)
+				(xy 46.0856 45.8480)
+				(xy 46.1337 45.9854)
+			) (stroke (width 0) (type solid)) (fill solid) (layer "F.Cu"))
 )
