File: PCB/solar-glow-drh-v2_1.kicad_sch (KiCad schematic)
At the start: 50 parts, among them J1 UPDI hdr, Q1 BCP5316MTWG, SW2 LED master, U1 AVR64DD28 (VQFN28), U2 ALD910025SAL, U3 LIS2DH12, U4 TLV431BCDBZR

Commit message: Add files via upload
Parts:
- PV1, PV2: value SM141K06L -> SM141K06TF
- U2: value ALD910025SAL -> ALD910025SALI
Changed lines of the file:
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@@
 			)
 		)
-		(property "Value" "ALD910025SAL"
+		(property "Value" "ALD910025SALI"
 			(at 91.01 129.54 0)
 			(show_name no)
@@
 			)
 		)
-		(property "Value" "SM141K06L"
+		(property "Value" "SM141K06TF"
 			(at 36.4 48.26 0)
 			(show_name no)
@@
 			)
 		)
-		(property "Value" "SM141K06L"
+		(property "Value" "SM141K06TF"
 			(at 36.4 78.74 0)
 			(show_name no)
