File: PCB/solar-glow-drh-v2_2.kicad_pcb (KiCad board)
At the start: 6 copper layers, 50.8 x 88.9 mm, 53 parts, among them J1 UPDI hdr, Q1 BCP5316MTWG, SW2 LED master, U1 AVR64DD28 (VQFN28), U2 ALD910025SAL, U3 LIS2DH12, U4 TLV431BCDBZR, U5 NT3H2211 NFC

Commit message: Add files via upload
Routing:
- net LA: track 212.6 -> 216.2 mm
- net LB: track 212.0 -> 213.7 mm
Changed lines of the file:
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@@
 	)
 	(via
-		(at 23.8 36.4)
+		(at 23.6 36.4)
 		(size 0.6)
 		(drill 0.3)
@@
 	(segment
 		(start 23.65 36.4)
-		(end 23.8 36.4)
+		(end 23.6 36.4)
 		(width 0.22)
 		(layer "B.Cu")
@@
 	)
 	(via
-		(at 16.03 34.96)
+		(at 16.7 34.96)
 		(size 0.6)
 		(drill 0.3)
@@
 	(segment
 		(start 16.95 34.96)
-		(end 16.03 34.96)
+		(end 16.51 34.96)
 		(width 0.22)
 		(layer "B.Cu")
@@
 	)
 	(segment
-		(start 9.606497 46.426031)
-		(end 10.230466 47.05)
+		(start 9.5 46.426)
+		(end 10.2305 47.05)
 		(width 0.16)
 		(layer "B.Cu")
@@
 	)
 	(segment
-		(start 9.156498 44.5)
-		(end 9.606497 44.949999)
+		(start 9.1565 44.5)
+		(end 9.5 44.95)
 		(width 0.16)
 		(layer "B.Cu")
@@
 	)
 	(segment
-		(start 9.606497 44.949999)
-		(end 9.606497 46.426031)
+		(start 9.5 44.95)
+		(end 9.5 46.426)
 		(width 0.16)
 		(layer "B.Cu")
@@
 	)
 	(via
-		(at 37.94 32.9)
+		(at 39 34)
 		(size 0.6)
 		(drill 0.3)
@@
 	)
 	(segment
+		(start 33.5 32)
+		(end 33.5 33.75)
+		(width 0.15)
+		(layer "B.Cu")
+		(net "LA")
+	)
+	(segment
 		(start 48.14 32.3)
 		(end 48.14 56.6)
@@
 	)
 	(segment
+		(start 33.5 33.75)
+		(end 34.1 33.75)
+		(width 0.15)
+		(layer "B.Cu")
+		(net "LA")
+	)
+	(segment
 		(start 48.14 56.6)
 		(end 37.64 56.6)
@@
 	)
 	(segment
-		(start 35.4 32.05)
-		(end 34.1 33.75)
+		(start 37.94 32.9)
+		(end 39 34)
 		(width 0.15)
 		(layer "B.Cu")
@@
 	(segment
 		(start 37.34 32)
-		(end 35.4 32.05)
+		(end 33.5 32)
 		(width 0.15)
 		(layer "B.Cu")
@@
 	)
 	(via
-		(at 35.45 33.05)
+		(at 34.55 32.5)
 		(size 0.6)
 		(drill 0.3)
@@
 	)
 	(segment
-		(start 35.45 33.05)
+		(start 34.55 32.5)
 		(end 34.55 33.3)
 		(width 0.15)
 		(layer "B.Cu")
-		(net "LB")
-	)
-	(segment
-		(start 36.2 32.6)
-		(end 35.45 33.05)
-		(width 0.15)
-		(layer "In3.Cu")
 		(net "LB")
 	)
@@
 	(segment
 		(start 37.34 32)
-		(end 36.2 32.6)
+		(end 34.55 32.5)
 		(width 0.15)
 		(layer "In3.Cu")
@@
 	(segment
 		(start 38.24 32.6)
-		(end 37.94 32.9)
-		(width 0.15)
-		(layer "In3.Cu")
+		(end 39 34)
+		(width 0.15)
+		(layer "In3.Cu")

Commit message: Add files via upload
Routing:
- net BTN: track 38.4 -> 0.00 mm, vias 3 -> 0
Changed lines of the file:
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@@
 		(net "PA4")
-	)
-	(segment
-		(start 25.4 57)
-		(end 25.4 55.8)
-		(width 0.22)
-		(layer "F.Cu")
-		(net "BTN")
-	)
-	(via
-		(at 6 40.7)
-		(size 0.4)
-		(drill 0.2)
-		(layers "F.Cu" "B.Cu")
-		(capping no)
-		(covering
-			(front no)
-			(back no)
-		)
-		(plugging
-			(front no)
-			(back no)
-		)
-		(filling no)
-		(net "BTN")
-	)
-	(via
-		(at 6.05 42.5)
-		(size 0.4)
-		(drill 0.2)
-		(layers "F.Cu" "B.Cu")
-		(capping no)
-		(covering
-			(front no)
-			(back no)
-		)
-		(plugging
-			(front no)
-			(back no)
-		)
-		(filling no)
-		(net "BTN")
-	)
-	(via
-		(at 25.4 57)
-		(size 0.6)
-		(drill 0.3)
-		(layers "F.Cu" "B.Cu")
-		(capping no)
-		(covering
-			(front no)
-			(back no)
-		)
-		(plugging
-			(front no)
-			(back no)
-		)
-		(filling no)
-		(net "BTN")
-	)
-	(segment
-		(start 7.5 40.5)
-		(end 6 40.7)
-		(width 0.16)
-		(layer "B.Cu")
-		(net "BTN")
-	)
-	(segment
-		(start 6.05 42.5)
-		(end 6.05 57)
-		(width 0.22)
-		(layer "In2.Cu")
-		(net "BTN")
-	)
-	(segment
-		(start 6.05 57)
-		(end 25.4 57)
-		(width 0.22)
-		(layer "In2.Cu")
-		(net "BTN")
-	)
-	(segment
-		(start 6 40.7)
-		(end 6.05 42.5)
-		(width 0.22)
-		(layer "In3.Cu")
-		(net "BTN")
 	)
 	(via
@@
 	)
 	(via
-		(at 34.55 32.5)
+		(at 34.55 32.6)
 		(size 0.6)
 		(drill 0.3)
@@
 	)
 	(segment
-		(start 34.55 32.5)
+		(start 34.55 32.6)
 		(end 34.55 33.3)
 		(width 0.15)
@@
 	(segment
 		(start 37.34 32)
-		(end 34.55 32.5)
-		(width 0.15)
-		(layer "In3.Cu")
+		(end 34.55 32.6)
+		(width 0.15)
+		(layer "In3.Cu")

Commit message: Add files via upload
Routing:
- net VS: track 11.9 -> 14.4 mm
- net GND: track 15.3 -> 17.5 mm
Changed lines of the file:
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@@
+	)
+	(segment
+		(start 13.01 48.5)
+		(end 13.45 48.5)
+		(width 0.22)
+		(layer "B.Cu")
+		(net "GND")
 	)
 	(segment
@@
 	)
 	(segment
+		(start 8.11 50.4)
+		(end 8.55 50.4)
+		(width 0.22)
+		(layer "B.Cu")
+		(net "GND")
+	)
+	(segment
 		(start 20.75 35.65)
 		(end 20.75 35.15)
@@
 	)
 	(segment
+		(start 10.01 45.5)
+		(end 10.45 45.5)
+		(width 0.22)
+		(layer "B.Cu")
+		(net "GND")
+	)
+	(segment
 		(start 10.45 45.5)
 		(end 10.45 46.52)
@@
 	)
 	(segment
+		(start 10.01 36.6)
+		(end 10.45 36.6)
+		(width 0.22)
+		(layer "B.Cu")
+		(net "GND")
+	)
+	(segment
 		(start 8.35 52.6)
 		(end 8.35 53.62)
+		(width 0.22)
+		(layer "B.Cu")
+		(net "GND")
+	)
+	(segment
+		(start 7.91 52.6)
+		(end 8.35 52.6)
 		(width 0.22)
 		(layer "B.Cu")
@@
 	)
 	(segment
+		(start 22.19 36.4)
+		(end 21.5 36.4)
+		(width 0.22)
+		(layer "B.Cu")
+		(net "VS")
+	)
+	(segment
 		(start 20.75 36.15)
 		(end 21.5 36.4)
@@
 	)
 	(segment
+		(start 16.51 32.4)
+		(end 16.95 32.4)
+		(width 0.22)
+		(layer "B.Cu")
+		(net "VS")
+	)
+	(segment
 		(start 9.9 38.9)
 		(end 9.9 38.3)
@@
 		(start 16.95 34.96)
 		(end 16.51 34.96)
+		(width 0.22)
+		(layer "B.Cu")
+		(net "VS")
+	)
+	(segment
+		(start 32.06 48.6)
+		(end 32.5 48.6)
+		(width 0.22)
+		(layer "B.Cu")
+		(net "VS")
+	)
+	(segment
+		(start 8.99 36.6)
+		(end 8.55 36.6)
+		(width 0.22)
+		(layer "B.Cu")
+		(net "VS")
+	)
+	(segment
+		(start 8.99 45.5)
+		(end 8.55 45.5)
 		(width 0.22)
 		(layer "B.Cu")
@@
 		(net "VSENSE")
 	)
+	(segment
+		(start 7.09 50.4)
+		(end 6.65 50.4)
+		(width 0.22)
+		(layer "B.Cu")
+		(net "VSENSE")
+	)

Commit message: Add files via upload
Routing:
- net GND: track 17.5 -> 18.4 mm, vias 26 -> 33
- net VS: track 14.4 -> 15.3 mm, vias 19 -> 28
- net VINB: vias 1 -> 2
- net VIN: vias 2 -> 3
Other:
- board text removed: "GND"
- board text removed: "OFF"
- board text removed: "ON"
- board text removed: "PA4"
- board text removed: "PC0"
- board text removed: "PC1"
- board text removed: "SCL"
- board text removed: "SDA"
- board text removed: "TINY"
- board text removed: "UPDI"
- board text removed: "VS"

Commit message: Add files via upload
Routing:
- net FD: track 0.00 -> 5.56 mm
- net VSENSE: track 16.1 -> 19.0 mm
- net VS: track 15.3 -> 17.6 mm, vias 28 -> 31
- net GND: track 18.4 -> 20.7 mm, vias 33 -> 35
- net VINB: vias 2 -> 1
- net VIN: vias 3 -> 2

Commit message: Add files via upload
Routing:
- net SDA: track 32.0 -> 0.00 mm, vias 3 -> 0
- net SCL: track 23.5 -> 0.00 mm, vias 3 -> 0
- net PA4: track 19.8 -> 0.00 mm, vias 2 -> 0
- net PC0: track 15.2 -> 0.00 mm, vias 2 -> 0
- net PC1: track 13.0 -> 0.00 mm, vias 2 -> 0
- net VS: track 17.6 -> 19.1 mm
- net GND: vias 35 -> 33

Commit message: Add files via upload
Routing:
- net SDA: track 0.00 -> 38.6 mm, vias 0 -> 2
- net SCL: track 0.00 -> 35.9 mm, vias 0 -> 4
- net VIN: track 19.9 -> 34.9 mm
- net LA: track 216.2 -> 227.2 mm
- net CLREF: track 0.00 -> 8.91 mm
- net CLBASE: track 0.00 -> 6.40 mm
- net LB: track 213.6 -> 218.0 mm, vias 1 -> 2
- net VINB: track 12.1 -> 15.6 mm
- net MID: track 82.6 -> 84.5 mm, vias 6 -> 7

Commit message: Add files via upload
Routing:
- net VIN: track 34.9 -> 88.8 mm, vias 2 -> 3
- net MID: track 84.5 -> 104.9 mm
Changed lines of the file:
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@@
+		(net "VIN")
+	)
+	(via
+		(at 44.685 28.099)
+		(size 0.6)
+		(drill 0.3)
+		(layers "F.Cu" "B.Cu")
+		(net "VIN")
+	)
+	(segment
+		(start 4.335 49.999)
+		(end 5.835 41.149)
+		(width 0.2)
+		(layer "B.Cu")
 		(net "VIN")
 	)
@@
 	)
 	(segment
+		(start 6.885 35.899)
+		(end 19.035 29.899)
+		(width 0.2)
+		(layer "B.Cu")
+		(net "VIN")
+	)
+	(segment
 		(start 46.489 10.2)
 		(end 45.589 13.5)
+		(width 0.2)
+		(layer "B.Cu")
+		(net "VIN")
+	)
+	(segment
+		(start 39.285 29.899)
+		(end 44.685 28.099)
+		(width 0.2)
+		(layer "B.Cu")
+		(net "VIN")
+	)
+	(segment
+		(start 5.835 41.149)
+		(end 5.835 39.049)
+		(width 0.2)
+		(layer "B.Cu")
+		(net "VIN")
+	)
+	(segment
+		(start 19.035 29.899)
+		(end 39.285 29.899)
+		(width 0.2)
+		(layer "B.Cu")
+		(net "VIN")
+	)
+	(segment
+		(start 5.835 39.049)
+		(end 6.885 35.899)
 		(width 0.2)
 		(layer "B.Cu")
@@
 	)
 	(segment
+		(start 21.675 59.205)
+		(end 21.225 49.305)
+		(width 0.2)
+		(layer "B.Cu")
+		(net "MID")
+	)
+	(segment
 		(start 24.95 38.905)
 		(end 24.95 38.605)
@@
 		(width 0.2)
 		(layer "B.Cu")
+		(net "MID")
+	)
+	(segment
+		(start 21.225 49.305)
+		(end 24.075 39.255)
+		(width 0.2)
+		(layer "B.Cu")
