File: PCB/solar-glow-drh-v2_2.kicad_pcb (KiCad board)
At the start: 6 copper layers, 50.8 x 88.9 mm, 53 parts, among them J1 UPDI hdr, Q1 BCP5316MTWG, SW2 LED master, U1 AVR64DD28 (VQFN28), U2 ALD910025SAL, U3 LIS2DH12, U4 TLV431BCDBZR, U5 NT3H2211 NFC

Commit message: Add files via upload
Routing:
- net MID: track 104.9 -> 109.7 mm, vias 7 -> 9
- net VIN: track 88.8 -> 91.6 mm, vias 3 -> 2
- net SDA: track 38.6 -> 40.5 mm
- net SCL: track 35.9 -> 36.9 mm

Commit message: Add files via upload
Routing:
- net FD: track 5.56 -> 36.0 mm, vias 0 -> 2
Changed lines of the file:
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@@
 		(net "LDRV4")
+	)
+	(via
+		(at 31.8 37)
+		(size 0.6)
+		(drill 0.3)
+		(layers "F.Cu" "B.Cu")
+		(capping no)
+		(covering
+			(front no)
+			(back no)
+		)
+		(plugging
+			(front no)
+			(back no)
+		)
+		(filling no)
+		(net "FD")
+	)
+	(via
+		(at 7 40.9)
+		(size 0.4)
+		(drill 0.2)
+		(layers "F.Cu" "B.Cu")
+		(capping no)
+		(covering
+			(front no)
+			(back no)
+		)
+		(plugging
+			(front no)
+			(back no)
+		)
+		(filling no)
+		(net "FD")
 	)
 	(segment
@@
 		(net "FD")
 	)
+	(segment
+		(start 7.5 40.9)
+		(end 7 40.9)
+		(width 0.2)
+		(layer "B.Cu")
+		(net "FD")
+	)
+	(segment
+		(start 7.6 37.6)
+		(end 7.6 37.5)
+		(width 0.2)
+		(layer "In2.Cu")
+		(net "FD")
+	)
+	(segment
+		(start 7.5 37.7)
+		(end 7.6 37.6)
+		(width 0.2)
+		(layer "In2.Cu")
+		(net "FD")
+	)
+	(segment
+		(start 19.3 38)
+		(end 19.4 38.1)
+		(width 0.2)
+		(layer "In2.Cu")
+		(net "FD")
+	)
+	(segment
+		(start 18.3 37.1)
+		(end 19.2 38)
+		(width 0.2)
+		(layer "In2.Cu")
+		(net "FD")
+	)
+	(segment
+		(start 7.6 37.5)
+		(end 8 37.1)
+		(width 0.2)
+		(layer "In2.Cu")
+		(net "FD")
+	)
+	(segment
+		(start 19.4 38.1)
+		(end 23.7 38.1)
+		(width 0.2)
+		(layer "In2.Cu")
+		(net "FD")
+	)
+	(segment
+		(start 19.2 38)
+		(end 19.3 38)
+		(width 0.2)
+		(layer "In2.Cu")
+		(net "FD")
+	)
+	(segment
+		(start 7 40.9)
+		(end 7.5 40.4)
+		(width 0.2)
+		(layer "In2.Cu")
+		(net "FD")
+	)
+	(segment
+		(start 24.8 39.2)
+		(end 24.9 39.2)
+		(width 0.2)
+		(layer "In2.Cu")
+		(net "FD")
+	)
+	(segment
+		(start 26.1 39.3)
+		(end 28.4 37)
+		(width 0.2)
+		(layer "In2.Cu")
+		(net "FD")
+	)
+	(segment
+		(start 7.5 40.4)
+		(end 7.5 37.7)
+		(width 0.2)
+		(layer "In2.Cu")
+		(net "FD")
+	)
+	(segment
+		(start 24.9 39.2)
+		(end 25 39.3)
+		(width 0.2)
+		(layer "In2.Cu")
+		(net "FD")
+	)
+	(segment
+		(start 25.9 39.4)
+		(end 26 39.3)
+		(width 0.2)
+		(layer "In2.Cu")
+		(net "FD")
+	)
+	(segment
+		(start 28.4 37)
+		(end 31.8 37)
+		(width 0.2)
+		(layer "In2.Cu")
+		(net "FD")
+	)
+	(segment
+		(start 25.8 39.3)
+		(end 25.9 39.4)
+		(width 0.2)
+		(layer "In2.Cu")
+		(net "FD")
+	)
+	(segment
+		(start 8 37.1)
+		(end 18.3 37.1)
+		(width 0.2)
+		(layer "In2.Cu")
+		(net "FD")
+	)
+	(segment
+		(start 23.7 38.1)
+		(end 24.8 39.2)
+		(width 0.2)
+		(layer "In2.Cu")
+		(net "FD")
+	)
+	(segment
+		(start 25 39.3)
+		(end 25.8 39.3)
+		(width 0.2)
+		(layer "In2.Cu")
+		(net "FD")
+	)
+	(segment
+		(start 26 39.3)
+		(end 26.1 39.3)
+		(width 0.2)
+		(layer "In2.Cu")
+		(net "FD")
+	)

Commit message: Add files via upload
Routing:
- net MID: track 109.7 -> 96.8 mm, vias 9 -> 8
- net VIN: track 91.6 -> 87.3 mm, vias 2 -> 1
- net VSENSE: track 19.0 -> 19.5 mm
- net VS: vias 31 -> 30

Commit message: Add files via upload
Routing:
- net MID: track 96.8 -> 95.1 mm
- net VS: track 19.1 -> 17.6 mm
- net GND: track 20.7 -> 20.2 mm
Changed lines of the file:
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@@
-	)
-	(segment
-		(start 24.9 35.095)
-		(end 24.43 35.266)
-		(width 0.22)
-		(layer "B.Cu")
-		(net "GND")
 	)
 	(segment
@@
 	)
 	(segment
-		(start 35.261 61.039)
-		(end 34.061 59.839)
-		(width 0.2)
-		(layer "B.Cu")
-		(net "MID")
-	)
-	(segment
 		(start 34.061 59.839)
 		(end 34.061 52.939)
@@
 	)
 	(segment
-		(start 8.55 36.6)
-		(end 7.63 36.6)
+		(start 7.63 36.6)
+		(end 8.99 36.6)
 		(width 0.22)
 		(layer "B.Cu")
@@
 	)
 	(segment
-		(start 16.51 32.4)
-		(end 16.95 32.4)
-		(width 0.22)
-		(layer "B.Cu")
-		(net "VS")
-	)
-	(segment
 		(start 9.9 38.9)
 		(end 9.9 38.3)
@@
 	)
 	(segment
-		(start 16.95 32.4)
+		(start 16.51 32.4)
 		(end 17.87 32.4)
-		(width 0.22)
-		(layer "B.Cu")
-		(net "VS")
-	)
-	(segment
-		(start 16.95 34.96)
-		(end 16.51 34.96)
 		(width 0.22)
 		(layer "B.Cu")
@@
 	)
 	(segment
-		(start 24.9 36.365)
-		(end 24.43 36.536)
-		(width 0.22)
-		(layer "B.Cu")
-		(net "VS")
-	)
-	(segment
 		(start 35.5 33.75)
 		(end 36 33.75)
-		(width 0.22)
-		(layer "B.Cu")
-		(net "VS")
-	)
-	(segment
-		(start 8.99 36.6)
-		(end 8.55 36.6)
-		(width 0.22)
-		(layer "B.Cu")
-		(net "VS")
-	)
-	(segment
-		(start 24.9 37.635)
-		(end 24.43 37.806)
 		(width 0.22)
 		(layer "B.Cu")
@@
 	)
 	(segment
-		(start 46.9 72.05)
-		(end 47.05 72.05)
-		(width 0.2)
-		(layer "B.Cu")
-		(net "CLREF")
-	)
-	(segment
 		(start 46.04 72.95)
 		(end 46.04 73.55)
@@
 	)
 	(segment
-		(start 4.7 36)
-		(end 4.7 35.86)
-		(width 0.22)
-		(layer "B.Cu")
-		(net "UPDI")
-	)
-	(segment
 		(start 11.5 26)
 		(end 13.3 24)
@@
 	)
 	(segment
-		(start 37.34 32)
-		(end 33.5 32)
-		(width 0.15)
-		(layer "B.Cu")
-		(net "LA")
-	)
-	(segment
-		(start 37.34 32)
+		(start 33.5 32)
 		(end 48.44 32)
 		(width 0.15)

Commit message: Add files via upload
Parts:
- PV1, PV2: value SM141K06L -> SM141K06TF
- U2: value ALD910025SAL -> ALD910025SALI
- moved C9 0.29 mm to (32.0, 38.5)
Routing:
- net VSENSE: track 19.5 -> 16.3 mm
- net LA: track 227.2 -> 227.8 mm

Commit message: Add files via upload
Routing:
- net GND: vias 33 -> 32
Changed lines of the file:
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@@
-	)
-	(via
-		(at 31.1 38.9)
-		(size 0.6)
-		(drill 0.3)
-		(layers "F.Cu" "B.Cu")
-		(capping no)
-		(covering
-			(front no)
-			(back no)
-		)
-		(plugging
-			(front no)
-			(back no)
-		)
-		(filling no)
-		(net "GND")
 	)
 	(via
