File: PCB/solar-glow-drh-v2_2.kicad_pcb (KiCad board)
At the start: 6 copper layers, 50.8 x 88.9 mm, 53 parts, among them J1 UPDI hdr, Q1 BCP5316MTWG, SW2 LED master, U1 AVR64DD28 (VQFN28), U2 ALD910025SALI, U3 LIS2DH12, U4 TLV431BCDBZR, U5 NT3H2211 NFC

Commit message: Add files via upload
Parts:
- added U6: TPS22918, Package_TO_SOT_SMD:SOT-23-6, B.Cu at (7.50, 33.0)
- C4: value 100nF -> 1uF
- C5: value VSENSE filt -> 10nF
- C9: value DNP NP0 -> NP0_DNP
- R1, R2, R3, R4: value LED ballast -> 150R
- R12: value TINY ballast -> 220R
- R5, R6: value VSENSE div -> 1M
- SJ1: value VDDIO2 jmp -> 0R
- U5: value NT3H2211 NFC -> NT3H2211
Connections:
- C8 pad 1: VS -> VNFC
- U1 pad 5: unconnected-(U1-PA7-Pad5) -> NFC_EN
- U5 pad 6: VS -> VNFC
Routing:
- net VNFC: track 0.00 -> 41.3 mm, vias 0 -> 3
- net NFC_EN: track 0.00 -> 18.1 mm, vias 0 -> 3
- net VS: track 17.6 -> 26.8 mm
- net LA: track 227.8 -> 233.9 mm
- net SDA: track 40.7 -> 46.1 mm
- net VIN: track 87.6 -> 91.6 mm
- net GND: track 20.2 -> 22.1 mm, vias 32 -> 33
- net MID: track 95.1 -> 95.9 mm

Commit message: Add files via upload
Parts:
- moved U6 1.41 mm to (6.34, 32.2), turned to 90 degrees
Connections:
- U6 pad 1: VS -> VNFC
- U6 pad 2: GND -> VNFC
- U6 pad 5: VNFC -> GND
- U6 pad 6: VNFC -> VS
Routing:
- net NFC_EN: track 18.1 -> 15.3 mm
- net VNFC: track 41.3 -> 38.6 mm
- net GND: track 22.1 -> 19.9 mm
- net VS: track 26.8 -> 27.9 mm
