File: PCB/solar-glow-drh-v2_2.kicad_sch (KiCad schematic)
At the start: 53 parts, among them J1 UPDI hdr, Q1 BCP5316MTWG, SW2 LED master, U1 AVR64DD28 (VQFN28), U2 ALD910025SALI, U3 LIS2DH12, U4 TLV431BCDBZR, U5 NT3H2211

Commit message: Add files via upload
Parts:
- added U6: TPS22918, Package_TO_SOT_SMD:SOT-23-6, symbol solarglow:U6
Connections:
- net GND: now also U6.2 (GND)
- net VS: now also U6.1 (VIN); no longer C8.1, U5.6 (VCC)
- net NFC_EN: now reaches U1.5 (PA7)
- net NFC_EN: now also U6.3 (ON)
- new net VNFC: C8.1, U5.6 (VCC), U6.5 (QOD), U6.6 (VOUT)

Commit message: Add files via upload
Parts:
- C4: value 100nF -> 1uF
- C5: value VSENSE filt -> 10nF
- R1, R2, R3, R4: value LED ballast -> 150R
- R12: value TINY ballast -> 220R
- R5, R6: value VSENSE div -> 1M
- SJ1: value VDDIO2 jmp -> 0R

Commit message: Add files via upload
Connections:
- net GND: now also U6.5 (GND); no longer U6.2 (GND)
- net VNFC: now also U6.1 (VOUT), U6.2 (QOD); no longer U6.5 (QOD), U6.6 (VOUT)
- net VS: now also U6.6 (VIN); no longer U6.1 (VIN)
Changed lines of the file:
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@@
 		(at 604.52 100.33)
+	)
+	(bus_entry
+		(at 2.54 38.1)
+		(size 2.54 2.54)
+		(stroke
+			(width 0)
+			(type default)
+		)
 	)
 	(wire
