File: PCB/solar-glow-drh-v2_2.kicad_sch (KiCad schematic)
At the start: 54 parts, among them J1 UPDI hdr, Q1 BCP5316MTWG, SW2 LED master, U1 AVR64DD28 (VQFN28), U2 ALD910025SALI, U3 LIS2DH12, U4 TLV431BCDBZR, U5 NT3H2211, U6 TPS22918

Commit message: Add files via upload
Parts:
- removed U6: TPS22918, Package_TO_SOT_SMD:SOT-23-6, symbol solarglow:U6
- C4: value 1uF -> 100nF
- C5: value 10nF -> VSENSE filt
- R1, R2, R3, R4: value 150R -> LED ballast
- R12: value 220R -> TINY ballast
- R5, R6: value 1M -> VSENSE div
- SJ1: value 0R -> VDDIO2 jmp
Connections:
- net VNFC is gone; now on net VS: C8.1, U5.6 (VCC)
- net NFC_EN: no longer names the net of U1.5 (PA7)
