File: PCB/solar-glow-drh-v2_3.kicad_pcb (KiCad board)
At the start: 4 copper layers, 50.8 x 88.9 mm, 54 parts, among them J1 UPDI hdr, Q1 BCP5316MTWG, SW2 LED master, U1 AVR64DD28 (VQFN28), U2 ALD910025SALI, U3 LIS2DH12, U4 TLV431BCDBZR, U5 NT3H2211, U6 TPS22918

Commit message: Add files via upload
Routing:
- net GND: track 19.9 -> 45.0 mm
- net VS: track 27.9 -> 41.4 mm
Changed lines of the file:
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@@
 	)
 	(segment
+		(start 25.864 35.064)
+		(end 24.564 35.214)
+		(width 0.25)
+		(layer "B.Cu")
+		(net "GND")
+	)
+	(segment
 		(start 13.01 48.5)
 		(end 13.45 48.5)
@@
 	)
 	(segment
+		(start 8.514 49.358)
+		(end 8.464 53.508)
+		(width 0.25)
+		(layer "B.Cu")
+		(net "GND")
+	)
+	(segment
 		(start 47.3 68)
 		(end 47.8 68)
@@
 	)
 	(segment
+		(start 13.273 19.467)
+		(end 13.273 19.667)
+		(width 0.25)
+		(layer "In1.Cu")
+		(net "GND")
+	)
+	(segment
+		(start 23.114 50.204)
+		(end 29.314 48.004)
+		(width 0.25)
+		(layer "In1.Cu")
+		(net "GND")
+	)
+	(segment
+		(start 16.864 49.004)
+		(end 23.114 50.204)
+		(width 0.25)
+		(layer "In1.Cu")
+		(net "GND")
+	)
+	(segment
+		(start 29.314 48.004)
+		(end 29.614 48.054)
+		(width 0.25)
+		(layer "In1.Cu")
+		(net "GND")
+	)
+	(segment
+		(start 13.414 49.504)
+		(end 16.864 49.004)
+		(width 0.25)
+		(layer "In1.Cu")
+		(net "GND")
+	)
+	(segment
+		(start 12.623 16.867)
+		(end 13.273 19.467)
+		(width 0.25)
+		(layer "In1.Cu")
+		(net "GND")
+	)
+	(segment
 		(start 43.4 71.9)
 		(end 46.5 71.9)
@@
 	)
 	(segment
+		(start 10.414 47.088)
+		(end 11.314 46.938)
+		(width 0.25)
+		(layer "B.Cu")
+		(net "VS")
+	)
+	(segment
 		(start 19.25 36.15)
 		(end 20.75 36.15)
@@
 	)
 	(segment
+		(start 11.314 46.938)
+		(end 13.164 45.088)
+		(width 0.25)
+		(layer "B.Cu")
+		(net "VS")
+	)
+	(segment
 		(start 32.06 48.6)
 		(end 32.5 48.6)
@@
 	)
 	(segment
+		(start 13.9 15.6)
+		(end 14.15 14.35)
+		(width 0.25)
+		(layer "B.Cu")
+		(net "VS")
+	)
+	(segment
 		(start 10.40213 34.839)
 		(end 11.123567 34.839)
@@
 	)
 	(segment
+		(start 8.514 46.488)
+		(end 10.414 47.088)
+		(width 0.25)
+		(layer "B.Cu")
+		(net "VS")
+	)
+	(segment
 		(start 21.5 36.4)
 		(end 21.75 36.4)
@@
 	)
 	(segment
+		(start 14.15 14.35)
+		(end 14.15 7.65)
+		(width 0.25)
+		(layer "B.Cu")
+		(net "VS")
+	)
+	(segment
 		(start 10.860165 32.078999)
 		(end 9.849999 32.078999)
@@
 	)
 	(via
-		(at 6.75 42.6)
-		(size 0.6)
-		(drill 0.3)
-		(layers "F.Cu" "B.Cu")
-		(net "NFC_EN")
-	)
-	(via
-		(at 3.65 42.6)
-		(size 0.6)
-		(drill 0.3)
-		(layers "F.Cu" "B.Cu")
-		(net "NFC_EN")
-	)
-	(via
-		(at 5.3925 33.3375)
-		(size 0.6)
-		(drill 0.3)
-		(layers "F.Cu" "B.Cu")
-		(net "NFC_EN")
-	)
-	(segment
-		(start 6.75 41.65)
-		(end 6.75 42.6)
-		(width 0.15)
-		(layer "B.Cu")
-		(net "NFC_EN")
-	)
-	(segment
-		(start 7.5 41.3)
-		(end 7.1 41.3)
-		(width 0.15)
-		(layer "B.Cu")
-		(net "NFC_EN")
-	)
-	(segment
-		(start 7.1 41.3)
-		(end 6.75 41.65)
-		(width 0.15)
-		(layer "B.Cu")
-		(net "NFC_EN")
-	)
-	(segment
-		(start 6.75 42.6)
-		(end 3.65 42.6)
-		(width 0.15)
-		(layer "In1.Cu")
-		(net "NFC_EN")
-	)
-	(segment
-		(start 5.3925 33.5075)
-		(end 5.3925 33.3375)
-		(width 0.15)
-		(layer "In2.Cu")
-		(net "NFC_EN")
-	)
-	(segment
-		(start 3.65 42.6)
-		(end 3.65 34.7)
-		(width 0.15)
-		(layer "In2.Cu")
-		(net "NFC_EN")
-	)
-	(segment
-		(start 3.65 34.7)
-		(end 3.7 34.65)
-		(width 0.15)
-		(layer "In2.Cu")
-		(net "NFC_EN")
-	)
-	(segment
-		(start 3.7 34.65)
-		(end 4.25 34.65)
-		(width 0.15)
-		(layer "In2.Cu")
-		(net "NFC_EN")
-	)
-	(segment
-		(start 4.25 34.65)
-		(end 5.3925 33.5075)
-		(width 0.15)
-		(layer "In2.Cu")
-		(net "NFC_EN")
-	)
-	(via
 		(at 35.97 31.63)
 		(size 0.6)
@@
 	)
 	(via
+		(at 6.75 42.6)
+		(size 0.6)
+		(drill 0.3)
+		(layers "F.Cu" "B.Cu")
+		(net "NFC_EN")
+	)
+	(via
+		(at 3.65 42.6)
+		(size 0.6)
+		(drill 0.3)
+		(layers "F.Cu" "B.Cu")
+		(net "NFC_EN")
+	)
+	(via
+		(at 5.3925 33.3375)
+		(size 0.6)
+		(drill 0.3)
+		(layers "F.Cu" "B.Cu")
+		(net "NFC_EN")
+	)
+	(segment
+		(start 6.75 41.65)
+		(end 6.75 42.6)
+		(width 0.15)
+		(layer "B.Cu")
+		(net "NFC_EN")
+	)
+	(segment
+		(start 7.5 41.3)
+		(end 7.1 41.3)
+		(width 0.15)
+		(layer "B.Cu")
+		(net "NFC_EN")
+	)
+	(segment
+		(start 7.1 41.3)
+		(end 6.75 41.65)
+		(width 0.15)
+		(layer "B.Cu")
+		(net "NFC_EN")
+	)
+	(segment
+		(start 6.75 42.6)
+		(end 3.65 42.6)
+		(width 0.15)
+		(layer "In1.Cu")
+		(net "NFC_EN")
+	)
+	(segment
+		(start 5.3925 33.5075)
+		(end 5.3925 33.3375)
+		(width 0.15)
+		(layer "In2.Cu")
+		(net "NFC_EN")
+	)
+	(segment
+		(start 3.65 42.6)
+		(end 3.65 34.7)
+		(width 0.15)
+		(layer "In2.Cu")
+		(net "NFC_EN")
+	)
+	(segment
+		(start 3.65 34.7)
+		(end 3.7 34.65)
+		(width 0.15)
+		(layer "In2.Cu")
+		(net "NFC_EN")
+	)
+	(segment
+		(start 3.7 34.65)
+		(end 4.25 34.65)
+		(width 0.15)
+		(layer "In2.Cu")
+		(net "NFC_EN")
+	)
+	(segment
+		(start 4.25 34.65)
+		(end 5.3925 33.5075)
+		(width 0.15)
+		(layer "In2.Cu")
+		(net "NFC_EN")
+	)
+	(via
 		(at 34.75 34)
 		(size 0.6)
@@
 	)
 	(zone
-		(layers "In2.Cu")
-		(name "NFC_COIL_POUR_KEEPOUT")
-		(hatch edge 0.508)
-		(connect_pads
-			(clearance 0)
-		)
-		(min_thickness 0.2)
-		(keepout
-			(tracks allowed)
-			(vias allowed)
-			(pads allowed)
-			(copperpour not_allowed)
-			(footprints allowed)
-		)
-		(placement
-			(enabled no)
-			(sheetname "")
-		)
-		(fill
-			(thermal_gap 0.2)
-			(thermal_bridge_width 0.25)
-			(island_removal_mode 0)
-		)
-		(polygon
-			(pts
-				(xy 36.78 31.55) (xy 49 31.55) (xy 49 57.35) (xy 36.78 57.35)
-			)
-		)
-	)
-	(zone
 		(net "GND")
 		(layer "In1.Cu")
@@
 			)
 		)
+	)
+	(zone
+		(layer "In2.Cu")
+		(name "NFC_COIL_POUR_KEEPOUT")
+		(hatch edge 0.508)
+		(connect_pads
+			(clearance 0)
+		)
+		(min_thickness 0.2)
+		(keepout
+			(tracks allowed)
+			(vias allowed)
+			(pads allowed)
+			(copperpour not_allowed)
+			(footprints allowed)
+		)
+		(placement
+			(enabled no)
+			(sheetname "")
+		)
+		(fill
+			(thermal_gap 0.2)
+			(thermal_bridge_width 0.25)
+			(island_removal_mode 0)
+		)
+		(polygon
+			(pts
+				(xy 36.78 31.55) (xy 49 31.55) (xy 49 57.35) (xy 36.78 57.35)
+			)
+		)

Commit message: Add files via upload
Routing:
- net VS: track 41.4 -> 46.6 mm
Changed lines of the file:
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@@
 		(net "MID")
+	)
+	(segment
+		(start 30.1 35.095)
+		(end 25.9 36.37)
+		(width 0.25)
+		(layer "F.Cu")
+		(net "VS")
+	)
+	(segment
+		(start 30.878595 35.228937)
+		(end 30.1 35.095)
+		(width 0.25)
+		(layer "F.Cu")
+		(net "VS")
 	)
 	(via
