File: PCB/solar-glow-drh-v2_3.kicad_sch (KiCad schematic)
At the start: 54 parts, among them J1 UPDI hdr, Q1 BCP5316MTWG, SW2 LED master, U1 AVR64DD28 (VQFN28), U2 ALD910025SALI, U3 LIS2DH12, U4 TLV431BCDBZR, U5 NT3H2211, U6 TPS22918

Commit message: Add files via upload
Changed lines of the file:
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@@
 		(at 604.52 100.33)
-	)
-	(bus_entry
-		(at 2.54 38.1)
-		(size 2.54 2.54)
-		(stroke
-			(width 0)
-			(type default)
-		)
 	)
 	(wire
