File: PCB/solar-glow-drh-v3_0.kicad_sch (KiCad schematic)
At the start: 54 parts, among them J1 UPDI hdr, Q1 BCP5316MTWG, SW2 LED master, U1 AVR64DD28 (VQFN28), U2 ALD910025SALI, U3 LIS2DH12, U4 TLV431BCDBZR, U5 NT3H2211, U6 TPS22918

Commit message: Add files via upload
Parts:
- added R14: 100k, solarglow:R14, symbol solarglow:R14
Connections:
- net GND: now also U6.2 (GND), R14.2; no longer U6.5 (GND)
- net NFC_EN: now also R14.1
- net VNFC: now also U6.5 (QOD), U6.6 (VOUT); no longer U6.1 (VOUT), U6.2 (QOD)
- net VS: now also U6.1 (VIN); no longer U6.6 (VIN)
Changed lines of the file:
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@@
+	)
+	(symbol
+		(lib_id "solarglow:R14")
+		(at 685.8 69.85 0)
+		(unit 1)
+		(body_style 1)
+		(exclude_from_sim no)
+		(in_bom yes)
+		(on_board yes)
+		(in_pos_files yes)
+		(dnp no)
+		(property "Reference" "R14"
+			(at 697.23 69.85 0)
+			(show_name no)
+			(do_not_autoplace no)
+			(effects
+				(font
+					(size 1.27 1.27)
+				)
+			)
+		)
+		(property "Value" "100k"
+			(at 697.23 74.93 0)
+			(show_name no)
+			(do_not_autoplace no)
+			(effects
+				(font
+					(size 1.27 1.27)
+				)
+			)
+		)
+		(property "Footprint" "solarglow:R14"
+			(at 697.23 80.01 0)
+			(hide yes)
+			(show_name no)
+			(do_not_autoplace no)
+			(effects
+				(font
+					(size 1.27 1.27)
+				)
+			)
+		)
+		(property "Datasheet" ""
+			(at 685.8 69.85 0)
+			(hide yes)
+			(show_name no)
+			(do_not_autoplace no)
+			(effects
+				(font
+					(size 1.27 1.27)
+				)
+			)
+		)
+		(property "Description" ""
+			(at 685.8 69.85 0)
+			(hide yes)
+			(show_name no)
+			(do_not_autoplace no)
+			(effects
+				(font
+					(size 1.27 1.27)
+				)
+			)
+		)
+		(pin "1"
+		)
+		(pin "2"
+		)
+		(instances
+			(project "solar-glow-drh-v2_2"
+				(path "/bf17630f-b49b-49a7-9335-83fa0a7a44d0"
+					(reference "R14")
+					(unit 1)
+				)
+			)
+		)
 	)
 	(symbol
@@
 				)
 			)
+		)
+	)
+	(wire
+		(pts
+			(xy 685.8 69.85) (xy 680.72 69.85)
+		)
+		(stroke
+			(width 0)
+			(type default)
+		)
+	)
+	(wire
+		(pts
+			(xy 685.8 74.93) (xy 680.72 74.93)
+		)
+		(stroke
+			(width 0)
+			(type default)
+		)
+	)
+	(global_label "NFC_EN"
+		(shape bidirectional)
+		(at 680.72 69.85 0)
+		(effects
+			(font
+				(size 1 1)
+			)
+		)
+		(property "Intersheetrefs" "${INTERSHEET_REFS}"
+			(at 345.44 63.5 0)
+			(hide yes)
+			(show_name no)
+			(do_not_autoplace no)
+			(effects
+				(font
+					(size 1.27 1.27)
+				)
+			)
+		)
+	)
+	(global_label "GND"
+		(shape bidirectional)
+		(at 680.72 74.93 0)
+		(effects
+			(font
+				(size 1 1)
+			)
+		)
+		(property "Intersheetrefs" "${INTERSHEET_REFS}"
+			(at 345.44 63.5 0)
+			(hide yes)
+			(show_name no)
+			(do_not_autoplace no)
+			(effects
+				(font
+					(size 1.27 1.27)
+				)
+			)

Commit message: Add files via upload
Parts:
- added JP1: bench hdr, solarglow:JP1, symbol solarglow:JP1
- added TP1: VIN tp, solarglow:TP1, symbol solarglow:TP1
Connections:
- net GND: now also JP1.1
- net SCL: now also JP1.3
- net SDA: now also JP1.4
- net VIN: now also TP1.1
- net VS: now also JP1.2

Commit message: Add files via upload
Parts:
- C9: value NP0_DNP -> 82pF-NP0-trim
- L1: value 2.76uH -> 1.0uH
Changed lines of the file:
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@@
 			)
 		)
-		(property "Value" "2.76uH"
+		(property "Value" "1.0uH"
 			(at 571.5 149.86 0)
 			(show_name no)
@@
 			)
 		)
-		(property "Value" "NP0_DNP"
+		(property "Value" "82pF-NP0-trim"
 			(at 571.5 124.46 0)
 			(show_name no)

Commit message: Add files via upload
Parts:
- U4: value TLV431BCDBZR -> TLV3011BIDBVR
Connections:
- net CLBASE: no longer U4.2 (CATHODE)
- net CLREF: no longer U4.1 (REF)
- net GND: no longer U4.3 (ANODE)

Commit message: Add files via upload
Parts:
- R7: value 1.8M -> 1.82M

Commit message: Add files via upload
Connections:
- net CLBASE: now also U4.1 (OUT)
- net CLREF: now also U4.4 (IN-)
- net GND: now also U4.2 (V-)
- net REF_TIE: now also U4.3 (IN+), U4.5 (REF)
- net VS: now also U4.6 (V+)
Changed lines of the file:
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@@
 	(wire
 		(pts
-			(xy 139.7 38.1) (xy 134.62 38.1)
-		)
-		(stroke
-			(width 0)
-			(type default)
-		)
-	)
-	(wire
-		(pts
 			(xy 350.52 58.42) (xy 345.44 58.42)
 		)
@@
 	(wire
 		(pts
-			(xy 139.7 48.26) (xy 134.62 48.26)
-		)
-		(stroke
-			(width 0)
-			(type default)
-		)
-	)
-	(wire
-		(pts
 			(xy 209.55 58.42) (xy 204.47 58.42)
 		)
@@
 	(wire
 		(pts
-			(xy 139.7 43.18) (xy 134.62 43.18)
-		)
-		(stroke
-			(width 0)
-			(type default)
-		)
-	)
-	(wire
-		(pts
 			(xy 350.52 93.98) (xy 345.44 93.98)
 		)
@@
 	(global_label "CLREF"
 		(shape input)
-		(at 137.16 40.64 0)
+		(at 139.7 40.64 0)
 		(effects
 			(font
@@
 		)
 		(property "Intersheetrefs" "${INTERSHEET_REFS}"
-			(at 137.16 40.64 0)
+			(at 139.7 40.64 0)
 			(hide yes)
 			(show_name no)
@@
 	(global_label "REF_TIE"
 		(shape input)
-		(at 154.94 45.72 180)
+		(at 152.4 45.72 180)
 		(effects
 			(font
@@
 	(global_label "VS"
 		(shape input)
-		(at 154.94 50.8 180)
+		(at 152.4 50.8 180)
 		(effects
 			(font
@@
 	(global_label "CLBASE"
 		(shape input)
-		(at 154.94 40.64 180)
+		(at 152.4 40.64 180)
 		(effects
 			(font
@@
 	(global_label "GND"
 		(shape input)
-		(at 137.16 50.8 0)
+		(at 139.7 50.8 0)
 		(effects
 			(font
@@
 		)
 		(property "Intersheetrefs" "${INTERSHEET_REFS}"
-			(at 137.16 50.8 0)
+			(at 139.7 50.8 0)
 			(hide yes)
 			(show_name no)
@@
 	(global_label "REF_TIE"
 		(shape input)
-		(at 137.16 45.72 0)
+		(at 139.7 45.72 0)
 		(effects
 			(font
@@
 		)
 		(property "Intersheetrefs" "${INTERSHEET_REFS}"
-			(at 137.16 45.72 0)
+			(at 139.7 45.72 0)
 			(hide yes)
 			(show_name no)

Commit message: Add files via upload
Parts:
- added D10: MMSD301T1G, solarglow:D10, symbol solarglow:D10
- added D11: MMSD301T1G, solarglow:D11, symbol solarglow:D11
- R7: value 1.82M -> 6.81M
- R8: value 1M -> 3.74M
Connections:
- net VS: no longer U4.6 (V+)
- new net VCMP: U4.6 (V+)
Changed lines of the file:
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@@
 		)
 	)
-	(global_label "VS"
+	(global_label "VCMP"
 		(shape input)
 		(at 152.4 50.8 180)
@@
 			)
 		)
-		(property "Value" "1.82M"
+		(property "Value" "6.81M"
 			(at 150.7 99.06 0)
 			(show_name no)
@@
 	)
 	(symbol
+		(lib_id "solarglow:D10")
+		(at 120 25 0)
+		(unit 1)
+		(body_style 1)
+		(exclude_from_sim no)
+		(in_bom yes)
+		(on_board yes)
+		(in_pos_files yes)
+		(dnp no)
+		(property "Reference" "D10"
+			(at 131 30.08 0)
+			(show_name no)
+			(do_not_autoplace no)
+			(effects
+				(font
+					(size 1.27 1.27)
+				)
+			)
+		)
+		(property "Value" "MMSD301T1G"
+			(at 131 35.16 0)
+			(show_name no)
+			(do_not_autoplace no)
+			(effects
+				(font
+					(size 1.27 1.27)
+				)
+			)
+		)
+		(property "Footprint" "solarglow:D10"
+			(at 131 40.24 0)
+			(show_name no)
+			(do_not_autoplace no)
+			(effects
+				(font
+					(size 1.27 1.27)
+				)
+			)
+		)
+		(property "Datasheet" ""
+			(at 120 25 0)
+			(show_name no)
+			(do_not_autoplace no)
+			(effects
+				(font
+					(size 1.27 1.27)
+				)
+			)
+		)
+		(property "Description" ""
+			(at 120 25 0)
+			(show_name no)
+			(do_not_autoplace no)
+			(effects
+				(font
+					(size 1.27 1.27)
+				)
+			)
+		)
+		(pin "A"
+		)
+		(pin "K"
+		)
+		(instances
+			(project "solar-glow-drh-v3_0"
+				(path "/bf17630f-b49b-49a7-9335-83fa0a7a44d0"
+					(reference "D10")
+					(unit 1)
+				)
+			)
+		)
+	)
+	(symbol
+		(lib_id "solarglow:D11")
+		(at 120 45 0)
+		(unit 1)
+		(body_style 1)
+		(exclude_from_sim no)
+		(in_bom yes)
+		(on_board yes)
+		(in_pos_files yes)
+		(dnp no)
+		(property "Reference" "D11"
+			(at 131 50.08 0)
+			(show_name no)
+			(do_not_autoplace no)
+			(effects
+				(font
+					(size 1.27 1.27)
+				)
+			)
+		)
+		(property "Value" "MMSD301T1G"
+			(at 131 55.16 0)
+			(show_name no)
+			(do_not_autoplace no)
+			(effects
+				(font
+					(size 1.27 1.27)
+				)
+			)
+		)
+		(property "Footprint" "solarglow:D11"
+			(at 131 60.24 0)
+			(show_name no)
+			(do_not_autoplace no)
+			(effects
+				(font
+					(size 1.27 1.27)
+				)
+			)
+		)
+		(property "Datasheet" ""
+			(at 120 45 0)
+			(show_name no)
+			(do_not_autoplace no)
+			(effects
+				(font
+					(size 1.27 1.27)
+				)
+			)
+		)
+		(property "Description" ""
+			(at 120 45 0)
+			(show_name no)
+			(do_not_autoplace no)
+			(effects
+				(font
+					(size 1.27 1.27)
+				)
+			)
+		)
+		(pin "A"
+		)
+		(pin "K"
+		)
+		(instances
+			(project "solar-glow-drh-v3_0"
+				(path "/bf17630f-b49b-49a7-9335-83fa0a7a44d0"
+					(reference "D11")
+					(unit 1)
+				)
+			)
+		)
+	)
+	(global_label "VIN"
+		(shape bidirectional)
+		(at 114.92 25 0)
+		(effects
+			(font
+				(size 1 1)
+			)
+		)
+		(property "Intersheetrefs" "${INTERSHEET_REFS}"
+			(at 114.92 25 0)
+			(hide yes)
+			(show_name no)
+			(do_not_autoplace no)
+			(effects
+				(font
+					(size 1.27 1.27)
+				)
+			)
+		)
+	)
+	(global_label "VCMP"
+		(shape bidirectional)
+		(at 114.92 30.08 0)
+		(effects
+			(font
+				(size 1 1)
+			)
+		)
+		(property "Intersheetrefs" "${INTERSHEET_REFS}"
+			(at 114.92 30.08 0)
+			(hide yes)
+			(show_name no)
+			(do_not_autoplace no)
+			(effects
+				(font
+					(size 1.27 1.27)
+				)
+			)
+		)
+	)
+	(global_label "VINB"
+		(shape bidirectional)
+		(at 114.92 45 0)
+		(effects
+			(font
+				(size 1 1)
+			)
+		)
+		(property "Intersheetrefs" "${INTERSHEET_REFS}"
+			(at 114.92 45 0)
+			(hide yes)
+			(show_name no)
+			(do_not_autoplace no)
+			(effects
+				(font
+					(size 1.27 1.27)
+				)
+			)
+		)
+	)
+	(global_label "VCMP"
+		(shape bidirectional)
+		(at 114.92 50.08 0)
+		(effects
+			(font
+				(size 1 1)
+			)
+		)
+		(property "Intersheetrefs" "${INTERSHEET_REFS}"
+			(at 114.92 50.08 0)
+			(hide yes)
+			(show_name no)
+			(do_not_autoplace no)
+			(effects
+				(font
+					(size 1.27 1.27)
+				)
+			)
+		)
+	)
+	(symbol
 		(lib_id "solarglow:SB3")
 		(at 279.4 200.66 0)
@@
 			)
 		)
-		(property "Value" "1M"
+		(property "Value" "3.74M"
 			(at 150.7 119.38 0)
 			(show_name no)

Commit message: Add files via upload
Connections:
- net VCMP: now also D10.K, D11.K
- net VIN: now also D10.A
- net VINB: now also D11.A
