File: PCB/solar-glow-drh-v3_0.kicad_sch (KiCad schematic)
At the start: 59 parts, among them J1 UPDI hdr, Q1 BCP5316MTWG, SW2 LED master, U1 AVR64DD28 (VQFN28), U2 ALD910025SALI, U3 LIS2DH12, U4 TLV3011BIDBVR, U5 NT3H2211, U6 TPS22918

Commit message: Add files via upload
Parts:
- added C10: 100nF, solarglow:C10, symbol solarglow:C10
Connections:
- net GND: now also C10.2
- net VCMP: now also C10.1

Commit message: Add files via upload
Parts:
- added C11: 200nF, solarglow:C11, symbol solarglow:C11
- added C12: 100nF, solarglow:C12, symbol solarglow:C12
- U3: value LIS2DH12 -> ADXL367
Connections:
- net GND: now also U3.1 (SCLK), U3.11 (GND), C11.2, C12.2; no longer U3.5 (RES), U3.6 (GND)
- net INT1: now also U3.5 (INT1); no longer U3.12 (INT1)
- net INT2: now also U3.6 (INT2); no longer U3.11 (INT2)
- net SCL: now also U3.4 (CS/SCL); no longer U3.1 (SCL)
- net SDA: now also U3.2 (MOSI/SDA); no longer U3.4 (SDA)
- net VS: now also U3.12 (VDDIO), C12.1; no longer U3.2 (CS), U3.9 (Vdd)
- new net VREG: C11.1, U3.9 (VREG_OUT1)
