File: PCB/solar-glow-drh-v3_0.kicad_sch (KiCad schematic)
At the start: 62 parts, among them J1 UPDI hdr, Q1 BCP5316MTWG, SW2 LED master, U1 AVR64DD28 (VQFN28), U2 ALD910025SALI, U3 ADXL367, U4 TLV3011BIDBVR, U5 NT3H2211, U6 TPS22918

Commit message: Add files via upload
Parts:
- JP1: value bench hdr -> GND VS SCL SDA
- TP1: value VIN tp -> VIN
- U3: footprint solarglow:U3 -> Package_TO_SOT_SMD:ADXL367 CC-12-4_ADI
- U4: footprint solarglow:U4 -> Package_TO_SOT_SMD:SOT-23-6
Changed lines of the file:
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@@
 			)
 		)
-		(property "Footprint" "solarglow:U4"
+		(property "Footprint" "Package_TO_SOT_SMD:SOT-23-6"
 			(at 150.7 53.34 0)
 			(show_name no)
@@
 			)
 		)
-		(property "Datasheet" ""
+		(property "Datasheet" "tlv3011b.pdf"
 			(at 139.7 38.1 0)
 			(show_name no)
@@
 			)
 		)
-		(property "Value" "VIN tp"
+		(property "Value" "VIN"
 			(at 421.21 362.16 0)
 			(show_name no)
@@
 			)
 		)
-		(property "Footprint" "solarglow:U3"
+		(property "Footprint" "Package_TO_SOT_SMD:ADXL367 CC-12-4_ADI"
 			(at 361.52 53.34 0)
 			(show_name no)
@@
 			)
 		)
-		(property "Datasheet" ""
+		(property "Datasheet" "datasheets/adxl367.pdf"
 			(at 350.52 38.1 0)
 			(show_name no)
@@
 			)
 		)
-		(property "Value" "bench hdr"
+		(property "Value" "GND VS SCL SDA"
 			(at 421.21 332.16 0)
 			(show_name no)

Commit message: Add files via upload
Parts:
- added C13: 4.7uF, solarglow:C7, symbol solarglow:C11
Connections:
- net ANODE: now also C13.1
- net GND: now also C13.2
Changed lines of the file:
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@@
 	(wire
 		(pts
+			(xy 120 165) (xy 114.92 165)
+		)
+		(stroke
+			(width 0)
+			(type default)
+		)
+	)
+	(wire
+		(pts
 			(xy 139.7 88.9) (xy 134.62 88.9)
 		)
@@
 	(wire
 		(pts
+			(xy 120 170.08) (xy 114.92 170.08)
+		)
+		(stroke
+			(width 0)
+			(type default)
+		)
+	)
+	(wire
+		(pts
 			(xy 120.65 30.48) (xy 115.57 30.48)
 		)
@@
 		)
 	)
+	(global_label "GND"
+		(shape bidirectional)
+		(at 114.92 170.08 0)
+		(effects
+			(font
+				(size 1 1)
+			)
+		)
+		(property "Intersheetrefs" "${INTERSHEET_REFS}"
+			(at 114.92 170.08 0)
+			(hide yes)
+			(show_name no)
+			(do_not_autoplace no)
+			(effects
+				(font
+					(size 1.27 1.27)
+				)
+			)
+		)
+	)
 	(global_label "LDRV1"
 		(shape bidirectional)
@@
 		)
 	)
+	(global_label "ANODE"
+		(shape bidirectional)
+		(at 114.92 165 0)
+		(effects
+			(font
+				(size 1 1)
+			)
+		)
+		(property "Intersheetrefs" "${INTERSHEET_REFS}"
+			(at 114.92 165 0)
+			(hide yes)
+			(show_name no)
+			(do_not_autoplace no)
+			(effects
+				(font
+					(size 1.27 1.27)
+				)
+			)
+		)
+	)
 	(global_label "CLBASE"
 		(shape bidirectional)
@@
 					(unit 1)
 				)
+			)
+		)
+	)
+	(symbol
+		(lib_id "solarglow:C11")
+		(at 120 165 0)
+		(unit 1)
+		(body_style 1)
+		(exclude_from_sim no)
+		(in_bom yes)
+		(on_board yes)
+		(in_pos_files yes)
+		(dnp no)
+		(property "Reference" "C13"
+			(at 131 170.08 0)
+			(show_name no)
+			(do_not_autoplace no)
+			(effects
+				(font
+					(size 1.27 1.27)
+				)
+			)
+		)
+		(property "Value" "4.7uF"
+			(at 131 175.16 0)
+			(show_name no)
+			(do_not_autoplace no)
+			(effects
+				(font
+					(size 1.27 1.27)
+				)
+			)
+		)
+		(property "Footprint" "solarglow:C7"
+			(at 131 180.24 0)
+			(show_name no)
+			(do_not_autoplace no)
+			(effects
+				(font
+					(size 1.27 1.27)
+				)
+			)
+		)
+		(property "Datasheet" ""
+			(at 120 165 0)
+			(show_name no)
+			(do_not_autoplace no)
+			(effects
+				(font
+					(size 1.27 1.27)
+				)
+			)
+		)
+		(property "Description" ""
+			(at 120 165 0)
+			(show_name no)
+			(do_not_autoplace no)
+			(effects
+				(font
+					(size 1.27 1.27)
+				)
+			)
+		)
+		(pin "1"
+		)
+		(pin "2"
+		)
+		(instances
+			(project "solar-glow-drh-v3_0"
+				(path "/bf17630f-b49b-49a7-9335-83fa0a7a44d0"
+					(reference "C13")
+					(unit 1)
+				)

Commit message: Add files via upload
Other:
- moved on the sheet: C13
Changed lines of the file:
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@@
 	(wire
 		(pts
-			(xy 120 165) (xy 114.92 165)
+			(xy 120.65 165.1) (xy 115.57 165.1)
 		)
 		(stroke
@@
 	(wire
 		(pts
-			(xy 120 170.08) (xy 114.92 170.08)
+			(xy 120.65 170.18) (xy 115.57 170.18)
 		)
 		(stroke
@@
 	(global_label "GND"
 		(shape bidirectional)
-		(at 114.92 170.08 0)
+		(at 115.57 170.18 0)
 		(effects
 			(font
@@
 		)
 		(property "Intersheetrefs" "${INTERSHEET_REFS}"
-			(at 114.92 170.08 0)
+			(at 115.57 170.18 0)
 			(hide yes)
 			(show_name no)
@@
 	(global_label "ANODE"
 		(shape bidirectional)
-		(at 114.92 165 0)
+		(at 115.57 165.1 0)
 		(effects
 			(font
@@
 		)
 		(property "Intersheetrefs" "${INTERSHEET_REFS}"
-			(at 114.92 165 0)
+			(at 115.57 165.1 0)
 			(hide yes)
 			(show_name no)
@@
 			)
 		)
-		(property "Description" ""
+		(property "Description" "Comparator + 1.242V ref, open-drain, SOT-23-6"
 			(at 139.7 38.1 0)
 			(show_name no)
@@
 	(symbol
 		(lib_id "solarglow:C11")
-		(at 120 165 0)
+		(at 120.65 165.1 0)
 		(unit 1)
 		(body_style 1)
@@
 		(dnp no)
 		(property "Reference" "C13"
-			(at 131 170.08 0)
+			(at 131.65 170.18 0)
 			(show_name no)
 			(do_not_autoplace no)
@@
 		)
 		(property "Value" "4.7uF"
-			(at 131 175.16 0)
+			(at 131.65 175.26 0)
 			(show_name no)
 			(do_not_autoplace no)
@@
 		)
 		(property "Footprint" "solarglow:C7"
-			(at 131 180.24 0)
+			(at 131.65 180.34 0)
 			(show_name no)
 			(do_not_autoplace no)
@@
 		)
 		(property "Datasheet" ""
-			(at 120 165 0)
+			(at 120.65 165.1 0)
 			(show_name no)
 			(do_not_autoplace no)
@@
 		)
 		(property "Description" ""
-			(at 120 165 0)
+			(at 120.65 165.1 0)
 			(show_name no)
 			(do_not_autoplace no)

Commit message: Add files via upload
Parts:
- J1, JP1, SB1, SB2, SB3, SB4, SW2, TC1, TP1: now not fitted; now left out of the parts list
- MH1, MH2, MH3, MH4, PV1, PV2, SC1, SC2, SC3, SC4: now left out of the parts list
Changed lines of the file:
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@@
 		(body_style 1)
 		(exclude_from_sim no)
-		(in_bom yes)
+		(in_bom no)
 		(on_board yes)
 		(in_pos_files yes)
-		(dnp no)
+		(dnp yes)
 		(property "Reference" "TC1"
 			(at 421.21 124.46 0)
@@
 		(body_style 1)
 		(exclude_from_sim no)
-		(in_bom yes)
+		(in_bom no)
 		(on_board yes)
 		(in_pos_files yes)
-		(dnp no)
+		(dnp yes)
 		(property "Reference" "SB3"
 			(at 290.4 205.74 0)
@@
 		(body_style 1)
 		(exclude_from_sim no)
-		(in_bom yes)
+		(in_bom no)
 		(on_board yes)
 		(in_pos_files yes)
@@
 		(body_style 1)
 		(exclude_from_sim no)
-		(in_bom yes)
+		(in_bom no)
 		(on_board yes)
 		(in_pos_files yes)
@@
 		(body_style 1)
 		(exclude_from_sim no)
-		(in_bom yes)
+		(in_bom no)
 		(on_board yes)
 		(in_pos_files yes)
@@
 		(body_style 1)
 		(exclude_from_sim no)
-		(in_bom yes)
+		(in_bom no)
 		(on_board yes)
 		(in_pos_files yes)
-		(dnp no)
+		(dnp yes)
 		(property "Reference" "J1"
 			(at 421.21 99.06 0)
@@
 		(body_style 1)
 		(exclude_from_sim no)
-		(in_bom yes)
+		(in_bom no)
 		(on_board yes)
 		(in_pos_files yes)
-		(dnp no)
+		(dnp yes)
 		(property "Reference" "TP1"
 			(at 421.21 357.08 0)
@@
 		(body_style 1)
 		(exclude_from_sim no)
-		(in_bom yes)
+		(in_bom no)
 		(on_board yes)
 		(in_pos_files yes)
@@
 		(body_style 1)
 		(exclude_from_sim no)
-		(in_bom yes)
+		(in_bom no)
 		(on_board yes)
 		(in_pos_files yes)
@@
 		(body_style 1)
 		(exclude_from_sim no)
-		(in_bom yes)
+		(in_bom no)
 		(on_board yes)
 		(in_pos_files yes)
-		(dnp no)
+		(dnp yes)
 		(property "Reference" "SB4"
 			(at 290.4 266.7 0)
@@
 		(body_style 1)
 		(exclude_from_sim no)
-		(in_bom yes)
+		(in_bom no)
 		(on_board yes)
 		(in_pos_files yes)
@@
 		(body_style 1)
 		(exclude_from_sim no)
-		(in_bom yes)
+		(in_bom no)
 		(on_board yes)
 		(in_pos_files yes)
-		(dnp no)
+		(dnp yes)
 		(property "Reference" "SW2"
 			(at 290.4 287.02 0)
@@
 		(body_style 1)
 		(exclude_from_sim no)
-		(in_bom yes)
+		(in_bom no)
 		(on_board yes)
 		(in_pos_files yes)
@@
 		(body_style 1)
 		(exclude_from_sim no)
-		(in_bom yes)
+		(in_bom no)
 		(on_board yes)
 		(in_pos_files yes)
-		(dnp no)
+		(dnp yes)
 		(property "Reference" "SB2"
 			(at 290.4 144.78 0)
@@
 		(body_style 1)
 		(exclude_from_sim no)
-		(in_bom yes)
+		(in_bom no)
 		(on_board yes)
 		(in_pos_files yes)
-		(dnp no)
+		(dnp yes)
 		(property "Reference" "JP1"
 			(at 421.21 327.08 0)
@@
 		(body_style 1)
 		(exclude_from_sim no)
-		(in_bom yes)
+		(in_bom no)
 		(on_board yes)
 		(in_pos_files yes)
@@
 		(body_style 1)
 		(exclude_from_sim no)
-		(in_bom yes)
+		(in_bom no)
 		(on_board yes)
 		(in_pos_files yes)
@@
 		(body_style 1)
 		(exclude_from_sim no)
-		(in_bom yes)
+		(in_bom no)
 		(on_board yes)
 		(in_pos_files yes)
-		(dnp no)
+		(dnp yes)
 		(property "Reference" "SB1"
 			(at 290.4 83.82 0)
@@
 		(body_style 1)
 		(exclude_from_sim no)
-		(in_bom yes)
+		(in_bom no)
 		(on_board yes)
 		(in_pos_files yes)
