File: PCB/solar-glow-drh-v3_0.kicad_pcb (KiCad board)
At the start: 2 copper layers, 50.8 x 88.9 mm, 54 parts, among them J1 UPDI hdr, Q1 BCP5316MTWG, SW2 LED master, U1 AVR64DD28 (VQFN28), U2 ALD910025SALI, U3 LIS2DH12, U4 TLV431BCDBZR, U5 NT3H2211, U6 TPS22918

Commit message: Add files via upload
Routing:
- net VS: track 288.1 -> 267.9 mm
- net MID: track 121.0 -> 113.8 mm
- net SCL: track 55.3 -> 51.1 mm
- net GND: track 93.1 -> 89.2 mm
- net VNFC: track 36.8 -> 34.9 mm
- net LDRV4: track 40.7 -> 39.7 mm
- net SDA: track 54.8 -> 54.0 mm
- net INT2: track 11.0 -> 10.5 mm

Commit message: Add files via upload
Routing:
- net GND: track 89.2 -> 64.8 mm
- net VS: track 267.9 -> 267.2 mm
- net VSENSE: track 15.5 -> 14.9 mm

Commit message: Add files via upload
Parts:
- added R14: 100k, solarglow:R14, B.Cu at (4.39, 29.4)
Connections:
- U6 pad 1: VNFC -> VS
- U6 pad 2: VNFC -> GND
- U6 pad 5: GND -> VNFC
- U6 pad 6: VS -> VNFC
Routing:
- net VS: track 267.2 -> 278.4 mm
- net NFC_EN: track 12.1 -> 17.1 mm, vias 2 -> 4
- net GND: track 64.8 -> 60.3 mm, vias 24 -> 26
- net MID: track 113.8 -> 111.9 mm
- net VDDIO2: track 14.2 -> 12.5 mm
- net VNFC: track 34.9 -> 33.7 mm
- net SCL: track 51.1 -> 51.7 mm

Commit message: Add files via upload
Parts:
- added JP1: GND VS SCL SDA, solarglow:JP1, B.Cu at (48.4, 14.5)
- added TP1: VIN, solarglow:TP1, B.Cu at (48.4, 12.0)
Routing:
- net GND: track 60.3 -> 110.3 mm
- net SCL: track 51.7 -> 86.4 mm, vias 6 -> 7
- net SDA: track 53.9 -> 77.6 mm, vias 0 -> 2
- net VS: track 278.4 -> 282.4 mm
- net VIN: track 91.4 -> 94.2 mm

Commit message: Add files via upload
Parts:
- U4: value TLV431BCDBZR -> TLV3011BIDBVR; footprint solarglow:U4 -> Package_TO_SOT_SMD:SOT-23-6
- turned U4 to 90 degrees
Connections:
- U4 pad 1: CLREF -> CLBASE
- U4 pad 2: CLBASE -> GND
- U4 pad 3: GND -> REF_TIE
Routing:
- net REF_TIE: track 0.00 -> 2.42 mm
- net GND: track 110.3 -> 112.6 mm
- net CLBASE: track 6.66 -> 8.83 mm, vias 0 -> 2
- net VINB: track 15.6 -> 17.7 mm
- net CLREF: track 8.94 -> 9.72 mm

Commit message: Add files via upload
Parts:
- added D10: MMSD301T1G, solarglow:D1, B.Cu at (48.5, 60.5)
- added D11: MMSD301T1G, solarglow:D1, B.Cu at (47.2, 60.5)
- moved D9 0.75 mm to (45.8, 61.0)
Connections:
- U4 pad 6: VS -> VCMP
Routing:
- net VIN: track 94.2 -> 128.1 mm
- net VCMP: track 0.00 -> 6.94 mm, vias 0 -> 2
- net VINB: track 17.7 -> 21.8 mm
- net VS: track 282.4 -> 286.3 mm

Commit message: Add files via upload
Parts:
- added C10: 100nF, solarglow:C10, B.Cu at (48.5, 68.0)
- D10: footprint solarglow:D1 -> solarglow:D10
- D11: footprint solarglow:D1 -> solarglow:D11
Routing:
- net VCMP: track 6.94 -> 7.79 mm
