File: PCB/solar-glow-drh-v3_0.kicad_pcb (KiCad board)
At the start: 2 copper layers, 50.8 x 88.9 mm, 62 parts, among them J1 UPDI hdr, Q1 BCP5316MTWG, SW2 LED master, U1 AVR64DD28 (VQFN28), U2 ALD910025SALI, U3 ADXL367, U4 TLV3011BIDBVR, U5 NT3H2211, U6 TPS22918

Commit message: Add files via upload
Routing:
- net GND: track 124.6 -> 127.0 mm, vias 33 -> 35

Commit message: Add files via upload
Routing:
- net VS: track 292.5 -> 293.2 mm
- net GND: track 127.0 -> 127.6 mm

Commit message: Add files via upload
Parts:
- added C13: 4.7uF, solarglow:C7, B.Cu at (26.2, 50.0)
- moved C5 7.48 mm to (5.05, 45.5), turned to 90 degrees
- moved R5 5.12 mm to (6.00, 45.5), turned to -90 degrees
- moved R6 4.94 mm to (6.95, 45.5), turned to 90 degrees
- moved SB4 2.63 mm to (34.8, 49.4), turned to 180 degrees
- moved SB1 1.98 mm to (16.2, 50.0), turned to 180 degrees
- moved R1 1.58 mm to (16.1, 48.0)
- moved SB2 1.37 mm to (23.1, 50.9)
- moved R4 1.31 mm to (34.8, 48.3)
- moved SB3 1.20 mm to (28.7, 50.8), turned to 180 degrees
- moved C3 0.52 mm to (12.7, 48.0)
- moved U5 0.25 mm to (35.1, 34.0)
Routing:
- net GND: track 127.6 -> 80.5 mm, vias 35 -> 20
- net VIN: track 128.1 -> 121.2 mm
- net LDRV4: track 40.6 -> 37.0 mm
- net VSENSE: track 14.7 -> 11.8 mm
- net NFC_EN: track 17.1 -> 15.7 mm
- net VNFC: track 34.0 -> 35.3 mm
- net ANODE: track 42.7 -> 41.4 mm
- net LB: track 27.6 -> 28.9 mm
- net UPDI: track 28.5 -> 29.7 mm
- net K2: track 6.36 -> 5.11 mm
- net K5: track 6.36 -> 5.50 mm
- net SDA: track 79.1 -> 78.3 mm
- net LDRV2: track 23.5 -> 24.3 mm
- net VDDIO2: track 12.6 -> 11.8 mm
- net VS: track 293.2 -> 292.5 mm, vias 17 -> 16
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
Commit message: Add files via upload
Parts:
- U3: value ADXL367 -> (none)
- moved C9 3.71 mm to (35.7, 39.1), turned to 180 degrees
- moved C13 1.63 mm to (27.1, 48.6)
- moved C8 0.75 mm to (32.3, 34.8)
- moved R6 0.34 mm to (6.61, 45.5)
- moved R5 0.33 mm to (5.67, 45.5)
- moved C5 0.28 mm to (4.77, 45.5)
- moved R3 0.18 mm to (28.9, 49.6)
- moved SB3 0.18 mm to (28.8, 50.9)
- moved SB2 0.13 mm to (23.1, 50.7)
Routing:
- net GND: track 80.5 -> 62.8 mm, vias 20 -> 8
- net LA: track 387.6 -> 383.2 mm
- net ANODE: track 41.4 -> 45.0 mm
- net VSENSE: track 11.8 -> 8.74 mm
- net LDRV3: track 37.3 -> 40.1 mm
- net VS: track 292.5 -> 294.9 mm
- net LB: track 28.9 -> 27.1 mm
- net VNFC: track 35.3 -> 33.9 mm
- net LDRV2: track 24.3 -> 25.2 mm
- net LDRV4: track 37.0 -> 37.7 mm
- net UPDI: track 29.7 -> 30.3 mm

Commit message: Add files via upload
Parts:
- U3: value (none) -> ADXL367
Changed lines of the file:
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@@
 			)
 		)
-		(property "Value" ""
+		(property "Value" "ADXL367"
 			(at 0 0 90)
 			(unlocked yes)

Commit message: Add files via upload
Parts:
- moved SB1 2.11 mm to (17.6, 48.5), turned to -90 degrees
- moved SB3 1.77 mm to (30.4, 50.2), turned to 90 degrees
- moved SB2 1.03 mm to (23.9, 50.0), turned to -90 degrees
- moved SB4 0.31 mm to (35.0, 49.6)
- moved C13 0.16 mm to (26.9, 48.6)
- moved C11 0.09 mm to (21.5, 37.6)
- moved C12 0.08 mm to (18.3, 33.1)
Routing:
- net SCL: track 89.5 -> 91.6 mm
- net SDA: track 78.4 -> 79.5 mm
- net LDRV1: track 15.6 -> 14.6 mm
- net LDRV2: track 25.2 -> 24.6 mm
- net VS: track 294.9 -> 295.4 mm
- net GND: track 62.8 -> 63.1 mm, vias 8 -> 6

Commit message: Add files via upload
Routing:
- net VNFC: track 33.9 -> 50.2 mm
- net SDA: track 79.5 -> 70.8 mm
- net FD: track 35.7 -> 41.0 mm
- net SCL: track 91.6 -> 96.5 mm, vias 9 -> 7
- net GND: track 63.1 -> 67.2 mm, vias 6 -> 5
- net VS: track 295.4 -> 292.6 mm, vias 16 -> 13
- net VIN: track 121.2 -> 120.2 mm
- net VSENSE: track 8.74 -> 8.01 mm
- net INT1: track 13.3 -> 12.7 mm
