File: PCB/solar-glow-drh-v3_0.kicad_pcb (KiCad board)
At the start: 2 copper layers, 50.8 x 88.9 mm, 63 parts, among them J1 UPDI hdr, Q1 BCP5316MTWG, SW2 LED master, U1 AVR64DD28 (VQFN28), U2 ALD910025SALI, U3 ADXL367, U4 TLV3011BIDBVR, U5 NT3H2211, U6 TPS22918

Commit message: Add files via upload
Routing:
- net GND: track 67.2 -> 70.2 mm
- net SCL: track 96.5 -> 95.1 mm
- net VS: track 292.6 -> 291.7 mm
- net SDA: track 70.8 -> 70.1 mm
- net CLBASE: track 8.83 -> 8.19 mm
