File: PCB/solar-glow-drh-v3_0.kicad_pcb (KiCad board)
At the start: 2 copper layers, 50.8 x 88.9 mm, 63 parts, among them J1 UPDI hdr, Q1 BCP5316MTWG, SW2 LED master, U1 AVR64DD28 (VQFN28), U2 ALD910025SALI, U3 ADXL367, U4 TLV3011BIDBVR, U5 NT3H2211, U6 TPS22918

Commit message: PCB: fix C13 footprint id (solarglow:C7 -> C13) and C11 value (200nF -> 220nF)
Two board-file corrections from the PCB audit. Identifier/value strings only,
no copper/pad/geometry change. Verified by exact single-token git diff, real-C7
untouched (pcb 7364, sch 3147), and unchanged paren balance in both files.

C13 footprint id: the footprint carried the stale base-footprint string
"solarglow:C7" in both the .kicad_pcb block (uuid 355e5d4a) and the .kicad_sch
Footprint property, a leftover from when C13 was split off C7. Caps are named
per refdes (solarglow:C1..C12); there was no solarglow:C13 and a duplicated
solarglow:C7. Renamed C13's footprint id to solarglow:C13 in both files. Also
clears the CI BOM's bogus Footprint=C7 column for C13.

C11 value: MPN GRM155R71C224KA12D is 0.22 uF (220 nF) but the value field read
"200nF". Corrected the instance and the lib-symbol default to "220nF".

Not changed (audit conclusions): L1 was already 1.0uH; R5/R6 "VSENSE div" and
the other descriptive value labels are house style, not placeholders (the BOM
grouping fix is a KiBot group-by-MPN config change, handed off separately); the
origin NPTH_mech footprint carries real non-plated holes and is not a stray.

Co-Authored-By: Claude Opus 4.8 <noreply@anthropic.com>
Claude-Session: https://claude.ai/code/session_01PBK3zFENdvoGtn8yP7qPA8
Parts:
- C13: footprint solarglow:C7 -> solarglow:C13
Changed lines of the file:
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@@
 		(embedded_fonts no)
 	)
-	(footprint "solarglow:C7"
+	(footprint "solarglow:C13"
 		(layer "B.Cu")
 		(at 26.89 48.62 90)

Commit message: PCB: complete C11 value fix on the board side (footprint Value 200nF -> 220nF)
Follow-up to 5f7a1ed. That commit set C11 = 220nF in the schematic only, but the
CI BOM sources its Value column from the PCB footprint, which still read "200nF"
(the C13 footprint-id fix landed in the BOM because it was a pcb-side change; the
C11 value change was sch-only, so it did not). The regenerated BOM therefore
still showed 200nF. Corrected the PCB C11 footprint Value to 220nF so schematic
and board agree, matching the 0.22 uF / 220 nF MPN (GRM155R71C224KA12D).

Line-anchored single-token edit (pcb line 8026); only 200nF in the file; paren
balance unchanged; no geometry change.

Co-Authored-By: Claude Opus 4.8 <noreply@anthropic.com>
Claude-Session: https://claude.ai/code/session_01PBK3zFENdvoGtn8yP7qPA8
Parts:
- C11: value 200nF -> 220nF
Changed lines of the file:
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@@
 			)
 		)
-		(property "Value" "200nF"
+		(property "Value" "220nF"
 			(at 0 0 0)
 			(layer "F.Fab")
