File: PCB/solar-glow-drh-v3_0.kicad_pcb (KiCad board)
At the start: 2 copper layers, 50.8 x 88.9 mm, 63 parts, among them J1 UPDI hdr, Q1 BCP5316MTWG, SW2 LED master, U1 AVR64DD28 (VQFN28), U2 ALD910025SALI, U3 ADXL367, U4 TLV3011BIDBVR, U5 NT3H2211, U6 TPS22918

Commit message: Add files via upload
Parts:
- moved R9 8.77 mm to (48.2, 79.1), turned to -90 degrees
- moved C7 7.70 mm to (48.8, 82.4)
- moved D9 7.62 mm to (45.8, 68.6)
- moved U4 7.55 mm to (47.4, 75.5), turned to -90 degrees
- moved R7 6.44 mm to (48.2, 78.2), turned to -90 degrees
- moved R8 5.20 mm to (46.7, 78.7), turned to 0 degrees
- moved C10 4.86 mm to (48.0, 72.8), turned to 90 degrees
- moved Q1 3.43 mm to (47.9, 68.1)
- moved D10 3.41 mm to (48.6, 63.9)
- moved D11 3.36 mm to (47.3, 63.9)
Routing:
- net VCMP: track 7.79 -> 19.6 mm, vias 2 -> 4
- net CLBASE: track 8.19 -> 19.7 mm, vias 2 -> 3
- net VIN: track 120.5 -> 127.7 mm
- net CLREF: track 9.72 -> 2.80 mm
- net MID: track 112.1 -> 118.6 mm
- net VS: track 291.7 -> 286.2 mm
- net VINB: track 21.1 -> 17.3 mm, vias 1 -> 2
- net SDA: track 70.1 -> 66.3 mm
- net GND: track 70.2 -> 66.6 mm, vias 5 -> 12
- net SCL: track 95.1 -> 91.8 mm
- added copper zone on F.Cu, net GND

Commit message: Add files via upload
Parts:
- added ?: , , F.Cu at (2.92, 59.6)
- added ?: , , F.Cu at (47.7, 60.5)
- added ?: , , F.Cu at (2.88, 28.8)
- added ?: , , F.Cu at (47.8, 29.8)
- moved D11 4.08 mm to (44.0, 66.2)
- moved R14 2.37 mm to (4.36, 31.8)
- moved D10 2.05 mm to (47.1, 65.4), turned to 0 degrees
- moved U6 1.24 mm to (7.46, 31.7)
Routing:
- net MID: track 118.6 -> 130.4 mm
- net SCL: track 91.8 -> 96.4 mm
- net VS: track 286.2 -> 281.6 mm
- net VCMP: track 19.6 -> 23.6 mm
- net VIN: track 127.7 -> 131.3 mm
- net SDA: track 66.3 -> 68.7 mm
- net VNFC: track 50.2 -> 48.9 mm
- net NFC_EN: track 15.5 -> 14.2 mm
- net GND: track 66.6 -> 65.9 mm, vias 12 -> 14
