File: PCB/solar-glow-drh-v3_0.kicad_pcb (KiCad board)
At the start: 2 copper layers, 50.8 x 88.9 mm, 67 parts, among them J1 UPDI hdr, Q1 BCP5316MTWG, SW2 LED master, U1 AVR64DD28 (VQFN28), U2 ALD910025SALI, U3 ADXL367, U4 TLV3011BIDBVR, U5 NT3H2211, U6 TPS22918

Commit message: Add files via upload
Parts:
- moved C4 15.3 mm to (13.7, 36.9), turned to -90 degrees
- moved C6 9.91 mm to (12.8, 36.9), turned to -90 degrees
- moved R10 8.35 mm to (8.40, 35.9)
- moved R11 4.56 mm to (11.9, 37.0), turned to 90 degrees
- moved C11 3.84 mm to (17.8, 36.7), turned to 180 degrees
- moved R13 1.45 mm to (33.8, 37.1), turned to 180 degrees
Routing:
- net MID: track 130.4 -> 118.3 mm
- net SCL: track 96.4 -> 89.1 mm
- net VS: track 281.6 -> 274.9 mm, vias 13 -> 11
- net CLBASE: track 19.7 -> 23.8 mm
- net GND: track 65.9 -> 61.8 mm, vias 14 -> 12
- net FD: track 41.0 -> 37.2 mm
- net VREG: track 3.18 -> 1.36 mm
- net VCMP: track 23.6 -> 22.2 mm
- net INT2: track 14.0 -> 13.1 mm, vias 2 -> 0
- net VIN: track 131.3 -> 130.5 mm
- net K2: track 5.11 -> 5.62 mm

Commit message: Add files via upload
Routing:
- net VS: track 274.9 -> 273.8 mm
