File: PCB/solar-glow-drh-v4_0.kicad_pcb (KiCad board)
At the start: 2 copper layers, 50.8 x 88.9 mm, 65 parts, among them J1 UPDI hdr, Q1 BCP5316MTWG, SW2 LED master, U1 AVR64DD28 (VQFN28), U2 ALD910025SALI, U3 ADXL367, U4 TLV3011BIDBVR, U5 NT3H2211, U6 TPS22918

Commit message: Add files via upload
Parts:
- moved SB1 12.6 mm to (5.64, 50.2)
- moved R1 10.4 mm to (5.69, 49.0), turned to 180 degrees
- moved C3 7.04 mm to (5.69, 48.0), turned to 180 degrees
- moved R2 3.28 mm to (26.2, 52.4), turned to -90 degrees
- moved SW2 2.94 mm to (26.4, 50.4)
- moved SB2 2.82 mm to (27.4, 52.4), turned to 90 degrees
- moved C13 1.02 mm to (25.9, 48.5), turned to -90 degrees
Routing:
- net MID: track 129.4 -> 165.4 mm
- net VS: track 295.9 -> 276.6 mm
- net K2: track 5.62 -> 15.4 mm
- net UPDI: track 119.2 -> 112.3 mm
- net LDRV3: track 38.9 -> 44.1 mm
- net VDDIO2: track 6.93 -> 10.8 mm
- net SCL: track 88.6 -> 85.8 mm
- net LDRV2: track 27.7 -> 30.3 mm
- net K3: track 8.53 -> 10.7 mm
- net SDA: track 70.3 -> 68.3 mm
- net TINY: track 6.94 -> 5.76 mm
- net LDRV1: track 15.4 -> 14.4 mm
- net ANODE: track 45.4 -> 46.3 mm, vias 6 -> 5
- net GND: vias 13 -> 15
