File: PCB/solar-glow-drh-v4_0.kicad_pcb (KiCad board)
At the start: 2 copper layers, 50.8 x 88.9 mm, 67 parts, among them J1 UPDI hdr, SW2 LED master, U1 AVR64DD28 (VQFN28), U3 ADXL367, U5 NT3H2211, U6 TPS22918, U8 AEM10300, U9 TPS7A0233 (SOT23-5*)

Commit message: Add files via upload
Parts:
- moved C7 83.7 mm to (5.39, 10.7)
- moved FB1 69.3 mm to (1.98, 54.7), turned to 90 degrees
- moved CSTO 63.5 mm to (6.15, 55.7), turned to -90 degrees
- moved C24 63.4 mm to (5.44, 58.7), turned to -90 degrees
- moved C23 61.5 mm to (3.10, 57.8), turned to 180 degrees
- moved U9 61.5 mm to (4.00, 55.4), turned to -90 degrees
- moved R16 57.1 mm to (6.40, 58.7), turned to -90 degrees
- moved R15 55.3 mm to (2.70, 52.6)
- moved L2 52.1 mm to (25.0, 56.9), turned to -90 degrees
- moved U8 48.9 mm to (31.2, 54.0)
- moved CSRC 39.4 mm to (25.0, 55.0), turned to 90 degrees
- moved CINT 33.8 mm to (35.8, 54.5), turned to 90 degrees
- moved R17 32.6 mm to (35.8, 56.4), turned to -90 degrees
- moved C22 23.1 mm to (44.8, 17.5), turned to -90 degrees
- moved C11 2.78 mm to (25.0, 30.5), turned to 90 degrees
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Routing:
- net STO: track 0.00 -> 197.5 mm, vias 0 -> 10
- net VS: track 276.6 -> 135.6 mm, vias 11 -> 6
- net SRC: track 0.00 -> 121.9 mm, vias 0 -> 2
- net VIN: track 72.7 -> 0.00 mm, vias 1 -> 0
- net EN_STO_CH: track 0.00 -> 45.5 mm, vias 0 -> 4
- net CLBASE: track 24.4 -> 0.00 mm, vias 3 -> 0
- net VINB: track 20.5 -> 0.00 mm, vias 2 -> 0
- net VCMP: track 19.6 -> 0.00 mm, vias 4 -> 0
- net MID: track 165.4 -> 146.6 mm
- net STO_SNS: track 0.00 -> 18.5 mm, vias 0 -> 2
- net VINT: track 0.00 -> 18.3 mm
- net UPDI: track 112.3 -> 127.2 mm
- net SCL: track 85.8 -> 78.9 mm
- net LX_LOUT: track 0.00 -> 5.29 mm
- net SDA: track 68.3 -> 73.5 mm
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
Commit message: Add files via upload
Parts:
- moved C22 54.5 mm to (3.51, 53.1), turned to 0 degrees
- moved R15 0.60 mm to (2.70, 52.0)
Routing:
- net MID: track 146.6 -> 145.4 mm
- net UPDI: track 127.2 -> 128.4 mm
- net STO_SNS: track 18.5 -> 19.2 mm
- net GND: vias 18 -> 19
