File: PCB/solar-glow-drh-v4_0.kicad_pcb (KiCad board)
At the start: 2 copper layers, 50.8 x 88.9 mm, 67 parts, among them J1 UPDI hdr, SW2 LED master, U1 AVR64DD28 (VQFN28), U3 ADXL367, U5 NT3H2211, U6 TPS22918, U8 AEM10300, U9 TPS7A0233 (SOT23-5*)

Commit message: PCB: give the AEM bulk caps valid refdes (CSRC/CINT/CSTO -> C25/C26/C27)
KiCad's schematic loader rejects letters-only reference designators (they
have no prefix/number split), so the descriptive CSRC/CINT/CSTO names the
board carried made the synced schematic fail to load in KiCad 10:
"Malformed component reference `CSRC`". The PCB editor had tolerated them,
so this only surfaced once the parts entered the schematic.

Rename to the next free C-numbers in BOTH the board and the schematic so
they stay matched: CSRC->C25 (BUFSRC bulk), CINT->C26 (VINT), CSTO->C27
(STO bulk). Values still describe the role. PCB change is the refdes text
only, no geometry or routing. Netlist re-reconciled clean against the
board after the rename.

Co-Authored-By: Claude Opus 4.8 <noreply@anthropic.com>
Claude-Session: https://claude.ai/code/session_01PBK3zFENdvoGtn8yP7qPA8
Parts:
- renumbered CSRC to C25, CINT to C26, CSTO to C27
Changed lines of the file:
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@@
 		(layer "B.Cu")
 		(at 35.8 54.49 90)
-		(property "Reference" "CINT"
+		(property "Reference" "C26"
 			(at -2.55 0 90)
 			(layer "B.SilkS")
@@
 		(layer "B.Cu")
 		(at 25 55 90)
-		(property "Reference" "CSRC"
+		(property "Reference" "C25"
 			(at -2.55 0 90)
 			(layer "B.SilkS")
@@
 		(layer "B.Cu")
 		(at 6.1468 55.7276 -90)
-		(property "Reference" "CSTO"
+		(property "Reference" "C27"
 			(at -2.55 0 90)
 			(layer "B.SilkS")
