File: PCB/solar-glow-drh-v4_0.kicad_pcb (KiCad board)
At the start: 2 copper layers, 50.8 x 88.9 mm, 67 parts, among them J1 UPDI hdr, SW2 LED master, U1 AVR64DD28 (VQFN28), U3 ADXL367, U5 NT3H2211, U6 TPS22918, U8 AEM10300, U9 TPS7A0233 (SOT23-5*)

Commit message: Add files via upload
Connections:
- U8 pad 1: (no net) -> unconnected-(U8-ZMPP-Pad1)
- U8 pad 15: (no net) -> unconnected-(U8-STO_OVDIS-Pad15)
- U8 pad 16: (no net) -> unconnected-(U8-STO_RDY-Pad16)
- U8 pad 17: (no net) -> unconnected-(U8-STO_OVCH-Pad17)
- U8 pad 26: (no net) -> unconnected-(U8-ST_STO-Pad26)
- U9 pad 4: (no net) -> unconnected-(U9-NC-Pad4)
- U9 pad 6: (no net) -> unconnected-(U9-NC-Pad6)
Routing:
- net MID: track 145.4 -> 153.2 mm
- net VINT: track 18.3 -> 20.5 mm
- net ANODE: track 45.5 -> 43.4 mm
- net NFC_EN: track 47.7 -> 46.2 mm
- net EN_STO_CH: track 45.5 -> 46.8 mm
- net FD: track 42.4 -> 41.5 mm
- net UPDI: track 128.4 -> 127.6 mm
