File: PCB/solar-glow-drh-v4_0.kicad_pcb (KiCad board)
At the start: 2 copper layers, 50.8 x 88.9 mm, 67 parts, among them J1 UPDI hdr, SW2 LED master, U1 AVR64DD28 (VQFN28), U3 ADXL367, U5 NT3H2211, U6 TPS22918, U8 AEM10300, U9 TPS7A0233 (SOT23-5*)

Commit message: Add files via upload
Parts:
- added U7: MB85RC512TY, Package_SO:SOIC-8_3.9x4.9mm_P1.27mm, B.Cu at (28.1, 37.3)
- moved R11 1.72 mm to (28.6, 32.6)
- moved R10 0.30 mm to (31.2, 31.6)
Routing:
- net VNFC: track 46.4 -> 54.8 mm
- net SDA: track 74.1 -> 79.3 mm
- net SCL: track 78.9 -> 84.0 mm, vias 6 -> 7
- net VS: track 134.8 -> 133.6 mm
