File: PCB/solar-glow-drh-v4_0.kicad_pcb (KiCad board)
At the start: 2 copper layers, 50.8 x 88.9 mm, 68 parts, among them J1 UPDI hdr, SW2 LED master, U1 AVR64DD28 (VQFN28), U3 ADXL367, U5 NT3H2211, U6 TPS22918, U7 MB85RC512TY, U8 AEM10300, U9 TPS7A0233 (SOT23-5*)

Commit message: SCH/PCB: give C28 a loadable footprint; set L2/C25 to 0603 lands
C28 (FRAM decoupling) was dropped by Update-PCB (missing_footprint)
because its footprint field was solarglow:C1, which only exists embedded
in other footprints and is not in a loadable library (the project's
solarglow.pretty holds just the two SCHURTER lands, and there is no
fp-lib-table). Point C28 at the standard Capacitor_SMD:C_0402_1005Metric
so Update-PCB can instantiate it.

Set the two parts that take real 0603 lands:
  L2  -> Inductor_SMD:L_0603_1608Metric   value 10uH
  C25 -> Capacitor_SMD:C_0603_1608Metric  value 22uF
Board-side land swap + reroute stays a KiCad step; the board keeps the
0402 land for now and only the marker-stripped values are synced here.

Co-Authored-By: Claude Opus 4.8 <noreply@anthropic.com>
Claude-Session: https://claude.ai/code/session_01PBK3zFENdvoGtn8yP7qPA8
Parts:
- C25: value 22uF *0805 -> 22uF
- L2: value 10uH *IND-land -> 10uH
Changed lines of the file:
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@@
 			)
 		)
-		(property "Value" "22uF *0805"
+		(property "Value" "22uF"
 			(at 0 0 90)
 			(layer "F.Fab")
@@
 			)
 		)
-		(property "Value" "10uH *IND-land"
+		(property "Value" "10uH"
 			(at 0 0 90)
 			(layer "F.Fab")
