File: PCB/solar-glow-drh-v4_0.kicad_pcb (KiCad board)
At the start: 2 copper layers, 50.8 x 88.9 mm, 68 parts, among them J1 UPDI hdr, SW2 LED master, U1 AVR64DD28 (VQFN28), U3 ADXL367, U5 NT3H2211, U6 TPS22918, U7 MB85RC512TY, U8 AEM10300, U9 TPS7A0233 (SOT23-5*)

Commit message: Add files via upload
Parts:
- added C28: 100nF, Capacitor_SMD:C_0402_1005Metric, B.Cu at (33.0, 39.5)
- C25: footprint solarglow:C1 -> Capacitor_SMD:C_0603_1608Metric
- L2: footprint solarglow:C1 -> Inductor_SMD:L_0603_1608Metric
- moved L2 1.91 mm to (25.3, 58.8)
- moved C25 0.43 mm to (25.1, 55.4)
Routing:
- net STO: track 199.1 -> 192.4 mm
- net SRC: track 122.0 -> 126.3 mm
- net VS: track 133.6 -> 131.7 mm
- net LX_LOUT: track 5.29 -> 6.61 mm
- net LDRV1: track 13.7 -> 12.7 mm
- net VNFC: track 54.8 -> 55.7 mm
- net FD: track 41.5 -> 40.7 mm
- net SDA: track 79.3 -> 78.7 mm
- net LDRV2: track 33.3 -> 32.8 mm

Commit message: Add files via upload
Parts:
- moved L2 3.66 mm to (28.1, 56.5), turned to 0 degrees
Routing:
- net LX_LOUT: track 6.61 -> 2.30 mm
- net LX_LIN: track 5.00 -> 2.93 mm

Commit message: Add files via upload
Parts:
- C13: value 4.7uF -> 10uF; footprint solarglow:C13 -> Capacitor_SMD:C_0603_1608Metric
- C23: value 1uF -> 2.2uF
- C27: footprint solarglow:C1 -> Capacitor_SMD:C_0603_1608Metric
- C4: value 4.7uF -> 10uF; footprint solarglow:C4 -> Capacitor_SMD:C_0603_1608Metric
- moved C7 1.74 mm to (5.25, 12.4)
- moved C4 1.09 mm to (5.05, 10.6), turned to -90 degrees
- moved C13 0.37 mm to (26.0, 48.0), turned to 180 degrees
- moved C27 0.22 mm to (6.15, 56.0)
- moved L2 0.20 mm to (28.1, 56.7)
- moved U9 0.10 mm to (3.90, 55.4)
Routing:
- net VS: track 131.7 -> 129.5 mm
- net NFC_EN: track 46.5 -> 45.9 mm

Commit message: Add files via upload
Parts:
- L2: footprint Inductor_SMD:L_0603_1608Metric -> Inductor_SMD:L_1008_2520Metric
- moved SC4 0.89 mm to (35.6, 72.8)
- moved R2 0.41 mm to (25.3, 52.0)
- moved C25 0.40 mm to (25.1, 55.0)
- moved SB2 0.40 mm to (26.4, 52.0)
- moved L2 0.35 mm to (27.9, 56.9)
Routing:
- net LX_LOUT: track 2.03 -> 2.94 mm
