File: PCB/solar-glow-drh-v4_0.kicad_pcb (KiCad board)
At the start: 2 copper layers, 50.8 x 88.9 mm, 69 parts, among them J1 UPDI hdr, SW2 LED master, U1 AVR64DD28 (VQFN28), U3 ADXL367, U5 NT3H2211, U6 TPS22918, U7 MB85RC512TY, U8 AEM10300, U9 TPS7A0233 (SOT23-5*)

Commit message: Add files via upload
Parts:
- JP1: value GND VS SCL SDA -> GND STO SCL SDA
- moved L2 2.08 mm to (26.5, 58.5), turned to -90 degrees
- moved SC4 1.15 mm to (36.8, 72.8)
- moved SB3 0.23 mm to (30.7, 49.5)
- moved J1 0.15 mm to (4.55, 38.4), turned to -90 degrees
Routing:
- net STO: track 192.8 -> 181.8 mm
- net MID: track 149.3 -> 155.5 mm
- net LX_LOUT: track 2.94 -> 6.02 mm
- net LX_LIN: track 3.26 -> 4.32 mm
- net SRC: track 126.0 -> 126.9 mm
- net EN_STO_CH: track 46.3 -> 47.0 mm
- net GND: vias 21 -> 20
Other:
- board text added: "ENABLE"
- board text added: "SCL"
- board text added: "SDA"
- board text added: "SRC"
- board text added: "STO"
- board text added: "TINY MODE"
