File: PCB/solar-glow-drh-v4_0.kicad_pcb (KiCad board)
At the start: 2 copper layers, 50.8 x 88.9 mm, 69 parts, among them J1 UPDI hdr, SW2 LED master, U1 AVR64DD28 (VQFN28), U3 ADXL367, U5 NT3H2211, U6 TPS22918, U7 MB85RC512TY, U8 AEM10300, U9 TPS7A0233 (SOT23-5*)

Commit message: FB1 + 8-screw: implement the STO_LDO ferrite island; document 8 mounting holes
FB1 (a 0603 ferrite the BOM calls an "STO island feed filter") sat with both pads
shorted on STO -- non-functional. Implemented it as a series filter on the U9 LDO
input: new net STO_LDO = {FB1.2, U9.1, U9.3, C22.1}, with FB1.1 + everything else
staying on STO. That gives STO --FB1--> STO_LDO, with C22 (1 uF) as the filtered
LDO-input cap, isolating U9 from the AEM10300 DCDC switching ripple (matters
because the 28-pin MCU has no AVDD, so the ADC rides VS). Applied to BOTH the
schematic (4 global labels) and the board pads (name-only nets; verified sch and
board agree).

NOTE: the board copper is not yet re-routed -- the old STO traces still run to
those pads, so DRC will flag STO_LDO as unrouted / net-mismatched until the trace
between FB1.1/FB1.2 is cut and STO_LDO routed to U9/C22 (no zone is involved).
Tracked in TODO.md.

Mounting holes: the board has 8 M2 GND holes (4 corner MH1-4 + 4 panel-corner
MP1-4) and the shell screws into all 8, so the docs now say 8 (README, PCB/README,
design-notes). The gold-frame GND tie stays a 4-corner mechanism (MP1-4 are GND
but not on the front gold set), so those specific references keep "four corner".

Also: sync-checklist net list (STO_LDO), BOM FB1 function, design-notes FB1
rationale.

Co-Authored-By: Claude Opus 4.8 <noreply@anthropic.com>
Claude-Session: https://claude.ai/code/session_01PBK3zFENdvoGtn8yP7qPA8
Connections:
- C22 pad 1: STO -> STO_LDO
- FB1 pad 2: STO -> STO_LDO
- U9 pad 1: STO -> STO_LDO
- U9 pad 3: STO -> STO_LDO
Changed lines of the file:
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@@
 			(layers "B.Cu" "B.Mask" "B.Paste")
 			(roundrect_rratio 0.25)
-			(net "STO")
+			(net "STO_LDO")
 			(pinfunction "IN_1")
 			(pintype "passive")
@@
 			(layers "B.Cu" "B.Mask" "B.Paste")
 			(roundrect_rratio 0.25)
-			(net "STO")
+			(net "STO_LDO")
 			(pinfunction "EN_3")
 			(pintype "passive")
@@
 			(layers "B.Cu" "B.Mask" "B.Paste")
 			(roundrect_rratio 0.25)
-			(net "STO")
+			(net "STO_LDO")
 			(pinfunction "2_2")
 			(pintype "passive")
@@
 			(layers "B.Cu" "B.Mask" "B.Paste")
 			(roundrect_rratio 0.25)
-			(net "STO")
+			(net "STO_LDO")
 			(pinfunction "1_1")
 			(pintype "passive")
