File: PCB/solar-glow-drh-v4_0.kicad_pcb (KiCad board)
At the start: 2 copper layers, 50.8 x 88.9 mm, 69 parts, among them J1 UPDI hdr, SW2 LED master, U1 AVR64DD28 (VQFN28), U3 ADXL367, U5 NT3H2211, U6 TPS22918, U7 MB85RC512TY, U8 AEM10300, U9 TPS7A0233 (SOT23-5*)

Commit message: Add files via upload
Parts:
- moved C22 3.84 mm to (1.90, 56.6), turned to -90 degrees
- moved C1 0.51 mm to (10.8, 41.0)
- moved FB1 0.13 mm to (2.10, 54.6), turned to -90 degrees
Routing:
- net STO_LDO: track 0.00 -> 5.47 mm
- net STO: track 181.8 -> 180.8 mm, vias 10 -> 12
- net VS: track 129.1 -> 128.5 mm
- net SRC: track 126.9 -> 126.4 mm
- net UPDI: track 88.4 -> 89.0 mm

Commit message: Add files via upload
Parts:
- SC1, SC3: value WS17 1F 2.75V -> SS17 1.8F 2.75V
Routing:
- net MID: track 155.5 -> 166.0 mm
- net ANODE: track 41.7 -> 45.3 mm
- net STO: track 180.8 -> 181.8 mm
- net VDDIO2: track 11.6 -> 10.7 mm

Commit message: Add files via upload
Parts:
- R15, R16: footprint solarglow:C1 -> Resistor_SMD:R_0603_1608Metric
- moved R16 2.46 mm to (6.15, 61.2)
- moved R15 0.48 mm to (3.17, 52.1)
Routing:
- net STO_SNS: track 19.1 -> 20.4 mm

Commit message: Add files via upload
Parts:
- C22, C23: footprint solarglow:C1 -> Capacitor_SMD:C_0603_1608Metric
- C26: footprint solarglow:C1 -> Capacitor_SMD:C_0805_2012Metric
- C27: footprint Capacitor_SMD:C_0603_1608Metric -> Capacitor_SMD:C_0805_2012Metric
- R5: footprint solarglow:R5 -> Resistor_SMD:R_0603_1608Metric
- R6: footprint solarglow:R6 -> Resistor_SMD:R_0603_1608Metric
- moved C27 7.81 mm to (2.54, 49.0), turned to 90 degrees
- moved R16 5.40 mm to (6.15, 55.8)
- moved C23 2.31 mm to (5.37, 58.2), turned to 0 degrees
- moved C24 0.83 mm to (5.91, 59.4), turned to 180 degrees
- moved R5 0.83 mm to (48.1, 24.8)
- moved C26 0.74 mm to (35.7, 53.8), turned to -90 degrees
- moved C5 0.45 mm to (45.2, 24.5)
- moved C22 0.44 mm to (1.68, 57.0)
- moved R17 0.27 mm to (35.6, 56.6)
- moved R6 0.07 mm to (46.5, 24.8)
Routing:
- net STO: track 182.3 -> 175.9 mm, vias 12 -> 10
- net STO_SNS: track 20.4 -> 18.6 mm
- net SRC: track 126.4 -> 128.0 mm
- net VSENSE: track 56.6 -> 58.1 mm
- net VS: track 128.4 -> 129.7 mm
- net UPDI: track 89.4 -> 90.1 mm
- net VINT: track 21.1 -> 20.5 mm

Commit message: Add files via upload
Parts:
- U7: footprint Package_SO:SOIC-8_3.9x4.9mm_P1.27mm -> Package_DFN_QFN:DFN-8-1EP_6x5mm_P1.27mm_EP4x4mm
Routing:
- net EN_STO_CH: track 46.6 -> 45.7 mm
- net GND: vias 20 -> 22

Commit message: Add files via upload
Parts:
- SJ1: value 0R -> DNP (was 0R VDDIO2 tie)
- U1: value AVR64DD28 (VQFN28) -> AVR64EA28 (VQFN28)
- U6: value TPS22918 -> TPS22917
- moved U7 0.11 mm to (28.1, 37.4)
Routing:
- net SRC: track 128.0 -> 132.1 mm
