File: PCB/solar-glow-drh-v4_0.kicad_sch (KiCad schematic)
At the start: 73 parts, among them J1 UPDI hdr, Q2 BSS138LT1G, SW2 LED master, U1 AVR64EA28 (VQFN28), U3 ADXL367, U5 NT3H2211, U6 TPS22917, U7 MB85RC512TY, U8 AEM10300, U9 TPS7A0233 (SOT23-5*)

Commit message: Make every cart line resolve: a P/N is an identifier, not prose
The DigiKey upload could not find the UPDI Friend. The cart carried Adafruit's
own product number 5879; DigiKey resolves 1528-5879-ND. A bare manufacturer
code does not error at upload -- the line just silently vanishes.

The data fix is one field. The reason it could happen is three:

1. NO MPN FALLBACK. The cart writer fell back to the MPN whenever a line had no
   distributor P/N, which is precisely how an unresolvable identifier reached a
   checkout page looking fine. A line without a distributor P/N is now a defect
   reported by the generator, which CI already runs without `|| true`. Proven by
   stripping PRG1's P/N: rc=1, and the line is ABSENT from the cart rather than
   silently wrong.

2. CBL1 IS NOT A CART LINE. DigiKey stocks only the legless TC2030-MCP-NL; the
   legged cable is a Tag-Connect direct order. Emitting it would fail at upload
   or, worse, buy the wrong cable. Its supplier is None, so it lands on the
   readable page instead -- which also fixes a crash, since the one-off loop
   lacked the `if supplier` filter its per-board sibling had and put a None key
   into a sorted().

3. THE ONE-OFF TABLE NOW SHOWS THE DISTRIBUTOR P/N. It was the only buy table
   without that column -- the exact column that failed.

The same defect one field over: C26/C27 carried "187-CL21B106KOQNNNG (Mouser)"
as a Supplier P/N, in both the schematic and the board. The origin is legible --
BOM/README.md rendered that column as `{dist_pn} ({source})`, so a live
availability CELL was copied back into the field it derives from, the report's
own source annotation glued onto the part number. A generated display string
round-tripped into a source of truth.

It was invisible because C26/C27 sit on the assembly side, where PCBWay buys by
MPN and never reads the field. It was not harmless: the grouping key is (mpn,
supplier, dist_pn), so the suffix also split one 2-off capacitor into two 1-off
purchase lines.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
Parts:
- C26, C27: Supplier P/N 187-CL21B106KOQNNNG (Mouser) -> 187-CL21B106KOQNNNG
Changed lines of the file:
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@@
 			)
 		)
-		(property "Supplier P/N" "187-CL21B106KOQNNNG (Mouser)"
+		(property "Supplier P/N" "187-CL21B106KOQNNNG"
 			(at 459.74 372.11 0)
 			(hide yes)
@@
 			)
 		)
-		(property "Supplier P/N" "187-CL21B106KOQNNNG (Mouser)"
-			(at 459.74 372.11 0)
-			(hide yes)
+		(property "Supplier P/N" "187-CL21B106KOQNNNG"
+			(at 459.74 372.11 0)
+			(hide yes)

Commit message: Give the design a Manufacturer field, and feed the guard that was starving
check_stock's pick_match() treats the manufacturer as a HARD filter for
collision-prone MPNs -- short or all-numeric ones -- and mfr_ok()'s docstring
names the case exactly: "a bare '5879' is both the Adafruit programmer and a
Pomona test clip". The filter has been inert since the xlsx master carrying the
Mfr column was culled: load_lines() sent mfr="" for every line, and mfr_ok()
returns True on an empty manufacturer. Not bypassed -- starved. It published a
Pomona clip ($88.96, 0 in stock) as the UPDI Friend while the real part had 54.

The design now carries the fact itself.

SCHEMATIC: a hidden Manufacturer property on all 53 placed symbols that carry a
real MPN. Values are the distributor's own spelling, taken live and cross-checked
against the Mfr column of the last pre-cull availability table (BOM/README.md @
cc55f40) -- all 28 unique MPNs agreed. Collision-prone ones were filtered on the
historical manufacturer while deriving, so a wrong match could not bootstrap a
wrong name into the file.

BOARD: the same field mirrored onto all 53 footprints, which is what "Update PCB
from Schematic" does. Not optional -- DRC's schematic-parity check reported 53
footprint_symbol_field_mismatch violations against the schematic-only edit, and
the board already mirrors MPN / Supplier / Supplier P/N. Each field was cloned
from that footprint's own Supplier block, so it inherits the exact position,
layer, hide flag and effects (including the justify mirror B-side parts carry)
rather than a hand-built block that could differ per side. UUIDs are uuid5 of the
refdes, so regenerating is byte-identical instead of a fresh diff. Both files
were edited as text with their CRLF convention preserved, the discipline
scripts/mask_art.py already follows for the board.

PLUMBING: _sch_parts reads it, build() carries it, load_lines() passes it. A part
with an MPN and no manufacturer now FAILS build(), so the guard canno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
Parts:
- C1, C11, C12, C13, C22, C23, C24, C28, C29, C3, C4, C5, C6, C7, C8, FB1, L2: Manufacturer (none) -> Murata Electronics
- C25: Manufacturer (none) -> TDK
- C26, C27: Manufacturer (none) -> Samsung Electro-Mechanics
- C9: Manufacturer (none) -> Johanson Technology Inc.
- D2, D3, D4, D5: Manufacturer (none) -> ams-OSRAM USA INC.
- PV1, PV2: Manufacturer (none) -> ANYSOLAR Ltd
- Q2: Manufacturer (none) -> onsemi
- R1, R10, R11, R12, R14, R16, R17, R18, R2, R3, R4, R5, R6: Manufacturer (none) -> YAGEO
- R15: Manufacturer (none) -> Vishay Dale
- SC1, SC2, SC3, SC4: Manufacturer (none) -> SCHURTER Inc.
- U1: Manufacturer (none) -> Microchip Technology
- U3: Manufacturer (none) -> Analog Devices Inc.
- U5: Manufacturer (none) -> NXP USA Inc.
- U6, U9: Manufacturer (none) -> Texas Instruments
- U7: Manufacturer (none) -> RAMXEED
- U8: Manufacturer (none) -> e-peas

Commit message: Name the manufacturers the way they name themselves
The Manufacturer values landed as whatever the stocking distributor calls the
vendor, which is a mix of legal entities and regional arms: "ams-OSRAM USA INC.",
"NXP USA Inc.", "SCHURTER Inc.", "ANYSOLAR Ltd", "YAGEO". Those are DigiKey's
catalogue names, not the makers' names for themselves, and this field is read by a
human in three buy documents now.

Rule applied: the manufacturer's own name, with distributor entity/region suffixes
(Inc./Ltd/LLC/USA) dropped and shouty catalogue casing normalised. 44 values in
each file; the ones already correct (Microchip Technology, Texas Instruments,
Samsung Electro-Mechanics, RAMXEED, onsemi, TDK, e-peas) are listed in the map
anyway so it shows the whole picture rather than only the exceptions.

Schematic and board are edited in ONE pass. A rename in only one of them would
reopen the 53 footprint_symbol_field_mismatch violations that made the field a
two-file change in the first place.

THE RISK HERE IS NOT COSMETIC, so it was measured rather than reasoned about.
mfr_ok() matches by token overlap and pick_match() makes it a hard filter for
collision-prone MPNs -- rename SCHURTER Inc. to something sharing no token and the
all-numeric 3-153-438/440 stop being distinguishable from another vendor's part.
Captured every resolved distributor P/N before the edit, re-ran check_stock after,
and diffed: all 47 rows resolve to the identical part. 30 ok / 0 sub / 0 dead.

DRC 0 schematic parity issues, 0 unconnected. check_consistency 0/0.
Parts:
- C1, C11, C12, C13, C22, C23, C24, C28, C29, C3, C4, C5, C6, C7, C8, FB1, L2: Manufacturer Murata Electronics -> Murata
- C9: Manufacturer Johanson Technology Inc. -> Johanson Technology
- D2, D3, D4, D5: Manufacturer ams-OSRAM USA INC. -> ams-OSRAM
- PV1, PV2: Manufacturer ANYSOLAR Ltd -> ANYSOLAR
- R1, R10, R11, R12, R14, R16, R17, R18, R2, R3, R4, R5, R6: Manufacturer YAGEO -> Yageo
- R15: Manufacturer Vishay Dale -> Vishay
- SC1, SC2, SC3, SC4: Manufacturer SCHURTER Inc. -> SCHURTER
- U3: Manufacturer Analog Devices Inc. -> Analog Devices
- U5: Manufacturer NXP USA Inc. -> NXP Semiconductors
Changed lines of the file:
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@@
 			)
 		)
-		(property "Manufacturer" "Murata Electronics"
+		(property "Manufacturer" "Murata"
 			(at 459.74 372.11 0)
 			(hide yes)
@@
 			)
 		)
-		(property "Manufacturer" "Murata Electronics"
+		(property "Manufacturer" "Murata"
 			(at 459.74 372.11 0)
 			(hide yes)
@@
 			)
 		)
-		(property "Manufacturer" "YAGEO"
+		(property "Manufacturer" "Yageo"
 			(at 459.74 372.11 0)
 			(hide yes)
@@
 			)
 		)
-		(property "Manufacturer" "Murata Electronics"
+		(property "Manufacturer" "Murata"
 			(at 459.74 372.11 0)
 			(hide yes)
@@
 			)
 		)
-		(property "Manufacturer" "ams-OSRAM USA INC."
+		(property "Manufacturer" "ams-OSRAM"
 			(at 459.74 372.11 0)
 			(hide yes)
@@
 			)
 		)
-		(property "Manufacturer" "YAGEO"
+		(property "Manufacturer" "Yageo"
 			(at 459.74 372.11 0)
 			(hide yes)
@@
 			)
 		)
-		(property "Manufacturer" "Murata Electronics"
+		(property "Manufacturer" "Murata"
 			(at 459.74 372.11 0)
 			(hide yes)
@@
 			)
 		)
-		(property "Manufacturer" "ams-OSRAM USA INC."
+		(property "Manufacturer" "ams-OSRAM"
 			(at 459.74 372.11 0)
 			(hide yes)
@@
 			)
 		)
-		(property "Manufacturer" "Murata Electronics"
+		(property "Manufacturer" "Murata"
 			(at 459.74 372.11 0)
 			(hide yes)
@@
 			)
 		)
-		(property "Manufacturer" "Vishay Dale"
+		(property "Manufacturer" "Vishay"
 			(at 459.74 372.11 0)
 			(hide yes)
@@
 			)
 		)
-		(property "Manufacturer" "YAGEO"
+		(property "Manufacturer" "Yageo"
 			(at 459.74 372.11 0)
 			(hide yes)
@@
 			)
 		)
-		(property "Manufacturer" "Murata Electronics"
+		(property "Manufacturer" "Murata"
 			(at 459.74 372.11 0)
 			(hide yes)
@@
 			)
 		)
-		(property "Manufacturer" "YAGEO"
+		(property "Manufacturer" "Yageo"
 			(at 459.74 372.11 0)
 			(hide yes)
@@
 			)
 		)
-		(property "Manufacturer" "YAGEO"
+		(property "Manufacturer" "Yageo"
 			(at 459.74 372.11 0)
 			(hide yes)
@@
 			)
 		)
-		(property "Manufacturer" "Murata Electronics"
+		(property "Manufacturer" "Murata"
 			(at 459.74 372.11 0)
 			(hide yes)
@@
 			)
 		)
-		(property "Manufacturer" "YAGEO"
+		(property "Manufacturer" "Yageo"
 			(at 459.74 372.11 0)
 			(hide yes)
@@
 			)
 		)
-		(property "Manufacturer" "Murata Electronics"
+		(property "Manufacturer" "Murata"
 			(at 459.74 372.11 0)
 			(hide yes)
@@
 			)
 		)
-		(property "Manufacturer" "SCHURTER Inc."
+		(property "Manufacturer" "SCHURTER"
 			(at 459.74 372.11 0)
 			(hide yes)
@@
 			)
 		)
-		(property "Manufacturer" "YAGEO"
+		(property "Manufacturer" "Yageo"
 			(at 459.74 372.11 0)
 			(hide yes)
@@
 			)
 		)
-		(property "Manufacturer" "SCHURTER Inc."
+		(property "Manufacturer" "SCHURTER"
 			(at 459.74 372.11 0)
 			(hide yes)
@@
 			)
 		)
-		(property "Manufacturer" "Murata Electronics"
+		(property "Manufacturer" "Murata"
 			(at 459.74 372.11 0)
 			(hide yes)
@@
 			)
 		)
-		(property "Manufacturer" "NXP USA Inc."
+		(property "Manufacturer" "NXP Semiconductors"
 			(at 459.74 372.11 0)
 			(hide yes)
@@
 			)
 		)
-		(property "Manufacturer" "YAGEO"
+		(property "Manufacturer" "Yageo"
 			(at 459.74 372.11 0)
 			(hide yes)
@@
 			)
 		)
-		(property "Manufacturer" "YAGEO"
+		(property "Manufacturer" "Yageo"
 			(at 459.74 372.11 0)
 			(hide yes)
@@
 			)
 		)
-		(property "Manufacturer" "YAGEO"
+		(property "Manufacturer" "Yageo"
 			(at 934.72 391.16 0)
 			(hide yes)
@@
 			)
 		)
-		(property "Manufacturer" "ANYSOLAR Ltd"
+		(property "Manufacturer" "ANYSOLAR"
 			(at 459.74 372.11 0)
 			(hide yes)
@@
 			)
 		)
-		(property "Manufacturer" "Murata Electronics"
+		(property "Manufacturer" "Murata"
 			(at 459.74 372.11 0)
 			(hide yes)
@@
 			)
 		)
-		(property "Manufacturer" "Johanson Technology Inc."
+		(property "Manufacturer" "Johanson Technology"
 			(at 560.07 119.38 0)
 			(hide yes)
@@
 			)
 		)
-		(property "Manufacturer" "SCHURTER Inc."
+		(property "Manufacturer" "SCHURTER"
 			(at 459.74 372.11 0)
 			(hide yes)
@@
 			)
 		)
-		(property "Manufacturer" "YAGEO"
+		(property "Manufacturer" "Yageo"
 			(at 459.74 372.11 0)
 			(hide yes)
@@
 			)
 		)
-		(property "Manufacturer" "YAGEO"
+		(property "Manufacturer" "Yageo"
 			(at 459.74 372.11 0)
 			(hide yes)
@@
 			)
 		)
-		(property "Manufacturer" "Murata Electronics"
+		(property "Manufacturer" "Murata"
 			(at 459.74 372.11 0)
 			(hide yes)
@@
 			)
 		)
-		(property "Manufacturer" "Murata Electronics"
+		(property "Manufacturer" "Murata"
 			(at 459.74 372.11 0)
 			(hide yes)
@@
 			)
 		)
-		(property "Manufacturer" "Analog Devices Inc."
+		(property "Manufacturer" "Analog Devices"
 			(at 459.74 372.11 0)
 			(hide yes)
@@
 			)
 		)
-		(property "Manufacturer" "Murata Electronics"
+		(property "Manufacturer" "Murata"
 			(at 459.74 392.43 0)
 			(hide yes)
@@
 			)
 		)
-		(property "Manufacturer" "ams-OSRAM USA INC."
+		(property "Manufacturer" "ams-OSRAM"
 			(at 459.74 372.11 0)
 			(hide yes)
@@
 			)
 		)
-		(property "Manufacturer" "Murata Electronics"
+		(property "Manufacturer" "Murata"
 			(at 459.74 372.11 0)
 			(hide yes)
@@
 			)
 		)
-		(property "Manufacturer" "Murata Electronics"
+		(property "Manufacturer" "Murata"
 			(at 459.74 372.11 0)
 			(hide yes)
@@
 			)
 		)
-		(property "Manufacturer" "ams-OSRAM USA INC."
+		(property "Manufacturer" "ams-OSRAM"
 			(at 459.74 372.11 0)
 			(hide yes)
@@
 			)
 		)
-		(property "Manufacturer" "YAGEO"
+		(property "Manufacturer" "Yageo"
 			(at 459.74 372.11 0)
 			(hide yes)
@@
 			)
 		)
-		(property "Manufacturer" "Murata Electronics"
+		(property "Manufacturer" "Murata"
 			(at 459.74 372.11 0)
 			(hide yes)
@@
 			)
 		)
-		(property "Manufacturer" "ANYSOLAR Ltd"
+		(property "Manufacturer" "ANYSOLAR"
 			(at 459.74 372.11 0)
 			(hide yes)
@@
 			)
 		)
-		(property "Manufacturer" "Murata Electronics"
+		(property "Manufacturer" "Murata"
 			(at 459.74 372.11 0)
 			(hide yes)
@@
 			)
 		)
-		(property "Manufacturer" "SCHURTER Inc."
+		(property "Manufacturer" "SCHURTER"
 			(at 459.74 372.11 0)
 			(hide yes)

Commit message: Buy from Mouser wherever Mouser can supply it -- which is not everywhere
Asked whether the whole hand-buy could move to Mouser, since PRG1 forces a Mouser
order anyway. It cannot: Mouser does not carry the solar cells at all. Checked
three ways on 2026-08-03 -- zero hits for SM141K06TF, zero for ANYSOLAR, zero for
IXOLAR. PV1/PV2 stay at DigiKey and a DigiKey order exists either way, so
consolidation was never actually on the table.

What IS on the table is price and depth, so the movable lines moved:

  SC1/SC3  3-153-440   486-3-153-440-ND  $17.16 -> 693-3-153-440  $16.50
  SC2/SC4  3-153-438   486-3-153-438-ND  $16.69 -> 693-3-153-438  $16.69 (same)
  FER1     364006      732-5049-ND       $17.43 -> 710-364006     $13.18
                                          41 in stock -> 119

~$5.57 per board, and 3x the ferrite depth on the one line whose DigiKey stock
(41) was the thinnest on the whole BOM. Same manufacturers, same MPNs.

SC1-4 live in the schematic + board, so both files are edited together as usual;
FER1 has no symbol and lives in OFF_BOARD. The edit is per-refdes, not a global
replace, because PV1/PV2 carry the same "DigiKey" string and must NOT be swept up
-- asserted in the applying script rather than eyeballed.

AND IT EXPOSED THE SAME BUG CLASS, MIRRORED. load_lines() never passed the
design's chosen supplier, so query_part was always DigiKey-first: after the move,
the availability table still reported SC1-4 and FER1 at DigiKey -- because DigiKey
stocks them -- while the cart CSVs beside it said Mouser. That is exactly the
disagreement this file was fixed for on 2026-08-02, running the other way (then
the buy list said DigiKey and the table said Mouser, and the table was right). The
table now asks the design's distributor first. Fallback is unchanged: a dry
preferred source still loses to a live other one, which is the C26/C27 rule and
the reason PRG1 was found in the first place.

Knock-on caught by the same run: FER1's datasheet filename embeds a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
Parts:
- SC1, SC3: Supplier DigiKey -> Mouser; Supplier P/N 486-3-153-440-ND -> 693-3-153-440
- SC2, SC4: Supplier DigiKey -> Mouser; Supplier P/N 486-3-153-438-ND -> 693-3-153-438
Changed lines of the file:
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@@
 			)
 		)
-		(property "Supplier" "DigiKey"
+		(property "Supplier" "Mouser"
 			(at 459.74 372.11 0)
 			(hide yes)
@@
 			)
 		)
-		(property "Supplier P/N" "486-3-153-438-ND"
+		(property "Supplier P/N" "693-3-153-438"
 			(at 459.74 372.11 0)
 			(hide yes)
@@
 			)
 		)
-		(property "Supplier" "DigiKey"
+		(property "Supplier" "Mouser"
 			(at 459.74 372.11 0)
 			(hide yes)
@@
 			)
 		)
-		(property "Supplier P/N" "486-3-153-440-ND"
+		(property "Supplier P/N" "693-3-153-440"
 			(at 459.74 372.11 0)
 			(hide yes)
@@
 			)
 		)
-		(property "Supplier" "DigiKey"
+		(property "Supplier" "Mouser"
 			(at 459.74 372.11 0)
 			(hide yes)
@@
 			)
 		)
-		(property "Supplier P/N" "486-3-153-440-ND"
+		(property "Supplier P/N" "693-3-153-440"
 			(at 459.74 372.11 0)
 			(hide yes)
@@
 			)
 		)
-		(property "Supplier" "DigiKey"
+		(property "Supplier" "Mouser"
 			(at 459.74 372.11 0)
 			(hide yes)
@@
 			)
 		)
-		(property "Supplier P/N" "486-3-153-438-ND"
+		(property "Supplier P/N" "693-3-153-438"
 			(at 459.74 372.11 0)
 			(hide yes)
