File: PCB/solar-glow-drh-v4_0.kicad_sch (KiCad schematic)
At the start: 73 parts, among them J1 UPDI hdr, Q2 BSS138LT1G, SW2 LED master, U1 AVR64EA28 (VQFN28), U3 ADXL367, U5 NT3H2211, U6 TPS22919, U7 MB85RC512TY, U8 AEM10300, U9 TPS7A0233 (SOT23-5*)

Commit message: Add files via upload
Parts:
- U9: value TPS7A0233 (SOT23-5*) -> TTPS7A0233PDQNR (X2SON-4); footprint solarglow:U9_SOT23_5 -> Package_SON:Texas_X2SON-4_1x1mm_P0.65mm
Connections:
- net GND: now also U9.5 (GND)
- net STO_LDO: no longer U9.1 (IN)
- net VS: now also U9.1 (OUT); no longer U9.5 (OUT)
Changed lines of the file:
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@@
 		)
 	)
-	(global_label "VS"
+	(global_label "GND"
 		(shape bidirectional)
 		(at 485.14 392.43 0)
@@
 		)
 	)
-	(global_label "STO_LDO"
-		(shape passive)
+	(global_label "VS"
+		(shape bidirectional)
 		(at 485.14 372.11 0)
 		(effects
@@
 			)
 		)
-		(property "Value" "TPS7A0233 (SOT23-5*)"
+		(property "Value" "TTPS7A0233PDQNR  (X2SON-4)"
 			(at 501.65 377.19 0)
 			(show_name no)
@@
 			)
 		)
-		(property "Footprint" "solarglow:U9_SOT23_5"
+		(property "Footprint" "Package_SON:Texas_X2SON-4_1x1mm_P0.65mm"
 			(at 501.65 382.27 0)
 			(hide yes)
